File: eagle/projects/comms_main_board/Comms_Main.sch (EAGLE design)
At the start: 53 parts, among them J1 RECE-20279-001E, Q1 CSD17579Q3A, U1 TPS562209DDCT, U2 LP2985-33DBVR, U3 LP5900TLX-3.3/NOPB, U4 TPS562209DDCT, U5 LMZ34002RKGR, U6 LM3488MMX/NOPB

Commit message: Finishing touches to GPS schematic
Parts:
- added LED1: (no value), comms:LEDCHIP-LED0805
- added R17: 100, comms:RES_0R100_0603
- added R18, R19, R20: 0.03, comms:RES_0RS030_0805
Connections:
- removed net 3P3V_ACC: R14.2, R15.2
- new net N$23: R17.1, U$1.4_TIMEPULSE
- new net N$25: LED1.A, R17.2
- new net N$26: U$1.3_RXD1
- new net N$27: R20.1, U$1.2_TXD1
- new net N$28: R18.1, U$1.9_V_RESET
- net 3P3V_SENSORS: now also R14.2, R15.2
- net GND: now also LED1.C
- net N$20: now also U$1.14_VCC_RF; no longer U$1.15_RESERVED
Other:
- note added: "COMMS MAX-M8Q Primary 2m GPS"
Changed lines of the file:
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@@
 <part name="C22" library="comms" deviceset="CAP" device="_0805" technology="_10NF0" value="10nF"/>
 <part name="L5" library="comms" deviceset="L" device="_0603" technology="_27NH0" value="27nH"/>
+<part name="R17" library="comms" deviceset="RES" device="_0603" technology="_0R100" value="100"/>
+<part name="LED1" library="comms" deviceset="LED" device="CHIP-LED0805"/>
+<part name="R19" library="comms" deviceset="RES" device="_0805" technology="_0RS030" value="0.03"/>
+<part name="R20" library="comms" deviceset="RES" device="_0805" technology="_0RS030" value="0.03"/>
+<part name="R18" library="comms" deviceset="RES" device="_0805" technology="_0RS030" value="0.03"/>
 </parts>
 <sheets>
@@
 <sheet>
 <plain>
+<text x="71.12" y="162.56" size="5.08" layer="91">COMMS MAX-M8Q Primary 2m GPS</text>
 </plain>
 <instances>
@@
 <instance part="C22" gate="G$1" x="76.2" y="78.74"/>
 <instance part="L5" gate="G$1" x="76.2" y="104.14"/>
+<instance part="R17" gate="G$1" x="177.8" y="96.52"/>
+<instance part="LED1" gate="G$1" x="193.04" y="96.52" rot="R90"/>
+<instance part="R19" gate="G$1" x="165.1" y="91.44"/>
+<instance part="R20" gate="G$1" x="177.8" y="86.36"/>
+<instance part="R18" gate="G$1" x="165.1" y="121.92"/>
 </instances>
 <busses>
@@
 <junction x="170.18" y="111.76"/>
 </segment>
-</net>
-<net name="3P3V_ACC" class="0">
 <segment>
 <pinref part="R15" gate="G$1" pin="2"/>
@@
 <wire x1="76.2" y1="76.2" x2="99.06" y2="76.2" width="0.1524" layer="91"/>
 <junction x="99.06" y="76.2"/>
+<pinref part="LED1" gate="G$1" pin="C"/>
+<wire x1="198.12" y1="96.52" x2="203.2" y2="96.52" width="0.1524" layer="91"/>
+<wire x1="203.2" y1="96.52" x2="203.2" y2="73.66" width="0.1524" layer="91"/>
+<wire x1="203.2" y1="73.66" x2="170.18" y2="73.66" width="0.1524" layer="91"/>
+<junction x="170.18" y="73.66"/>
 </segment>
 </net>
@@
 </segment>
 </net>
+<net name="N$23" class="0">
+<segment>
+<pinref part="U$1" gate="G$1" pin="4_TIMEPULSE"/>
+<pinref part="R17" gate="G$1" pin="1"/>
+<wire x1="157.48" y1="96.52" x2="172.72" y2="96.52" width="0.1524" layer="91"/>
+</segment>
+</net>
+<net name="N$25" class="0">
+<segment>
+<pinref part="R17" gate="G$1" pin="2"/>
+<pinref part="LED1" gate="G$1" pin="A"/>
+<wire x1="182.88" y1="96.52" x2="190.5" y2="96.52" width="0.1524" layer="91"/>
+</segment>
+</net>
+<net name="N$26" class="0">
+<segment>
+<pinref part="U$1" gate="G$1" pin="3_RXD1"/>
+<wire x1="157.48" y1="91.44" x2="162.56" y2="91.44" width="0.1524" layer="91"/>
+</segment>
+</net>
+<net name="N$27" class="0">
+<segment>
+<pinref part="U$1" gate="G$1" pin="2_TXD1"/>
+<pinref part="R20" gate="G$1" pin="1"/>
+<wire x1="157.48" y1="86.36" x2="172.72" y2="86.36" width="0.1524" layer="91"/>
+</segment>
+</net>
+<net name="N$28" class="0">
+<segment>
+<pinref part="U$1" gate="G$1" pin="9_V_RESET"/>
+<pinref part="R18" gate="G$1" pin="1"/>
+<wire x1="157.48" y1="121.92" x2="160.02" y2="121.92" width="0.1524" layer="91"/>
+</segment>
+</net>
 <net name="N$20" class="0">
 <segment>
+<pinref part="U$1" gate="G$1" pin="14_VCC_RF"/>
+<wire x1="111.76" y1="101.6" x2="106.68" y2="101.6" width="0.1524" layer="91"/>
+<wire x1="106.68" y1="101.6" x2="106.68" y2="96.52" width="0.1524" layer="91"/>
 <pinref part="R16" gate="G$1" pin="2"/>
-<pinref part="U$1" gate="G$1" pin="15_RESERVED"/>
-<wire x1="96.52" y1="96.52" x2="111.76" y2="96.52" width="0.1524" layer="91"/>
-</segment>
-</net>
+<wire x1="106.68" y1="96.52" x2="96.52" y2="96.52" width="0.1524" layer="91"/>
+</segment>
+</net>

Commit message: Pressure and Temp Sensor Schematics
Parts:
- added C23, C26, C27: 100nF, comms:CAP_100NF0_0603
- added R21, R22, R23, R24, R25, R26, R27, R28, R29, R30, R33, R34, R35: 0.0, comms:RES_0R0_0805
- added R31, R32, R36, R37: 4.7k, daqcs:RES_4R7_0603
- added U$2, U$3, U$4, U$5: PRT-12639, comms:PRT-12639
- added U7: PCT2075D,118, comms:PCT2075D,118SOIC8
- added U8: MS560702BA03-50, comms:MS5607-02BA03_8SMD
- R18, R19, R20: value 0.03 -> 0.0; device comms:RES_0RS030_0805 -> comms:RES_0R0_0805
Connections:
- new net N$29: R24.2, U$2.RING1
- new net N$30: R23.1, U$4.TIP
- new net N$31: R24.1, U$3.RING1
- new net N$32: R21.1, U$4.RING1
- new net N$33: R21.2, U$5.RING1
- new net N$34: R22.2, U$5.EARTH, U$5.RING2
- new net N$35: R23.2, U$5.TIP
- new net N$36: R25.2, U$2.TIP
- new net N$37: R27.2, U$3.EARTH, U$3.RING2
- new net N$38: R26.2, U$3.TIP
- new net N$39: R28.2, U7.A0
- new net N$40: R29.2, U7.A1
- new net N$41: R30.2, U7.A2
- new net N$42: R33.1, U7.OS
- new net N$43: R34.2, U8.CSB@1, U8.CSB@2
- new net N$46: R35.1, U8.SDO
- new net N$49: R35.2
- new net PRESS_SCL: U8.SCLK
- new net PRESS_SDA: R36.1, U8.SDI/SDA
- new net PTT: R27.1
- new net TEMP_OS: R33.2
- new net TEMP_SCL: R32.1, U7.SCL
- new net TEMP_SDA: R31.1, U7.SDA
- net 3P3V_SENSORS: now also C23.2, C26.2, C27.1, R31.2, R32.2, R36.2, R37.2, U7.VCC, U8.PS, U8.VDD
- net GND: now also C23.1, C26.1, C27.2, R22.1, R28.1, R29.1, R30.1, R34.1, U$2.EARTH, U$2.RING2, U$4.EARTH, U$4.RING2, U7.GND, U8.GND
- net N$22: now also L5.2
- net N$26: now also R19.1
Other:
- note added: "2m Transceiver"
- note added: "2m Transceiver -> Pi"
- note added: "COMMS 2m Transceiver Audio Jumpers"
- note added: "COMMS Sensors"
- note added: "Pi"
- note added: "Pi -> 2m Transceiver"
- note added: "Pressure Sensor"
- note added: "Temp Sensor"

Commit message: Changeess
Parts:
- added R38, R39: 0.0, comms:RES_0R0_0805
- renumbered U$1 to U9
Connections:
- new net N$44: R38.2, U9.13_ANTON
- new net N$45: R39.1, U9.5_EXTINT0
Other:
- moved on the sheet: R16
Changed lines of the file:
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@@
 <part name="L4" library="comms" deviceset="L" device="-680ML" technology="_68UH0" value="68uH"/>
 <part name="FRAME4" library="frames" deviceset="A4L-LOC" device=""/>
-<part name="U$1" library="comms" deviceset="UBLOX_MAX" device="" value="MAX-M8Q"/>
 <part name="R14" library="daqcs" deviceset="RES" device="_0603" technology="_4R7" value="4.7k"/>
 <part name="R15" library="daqcs" deviceset="RES" device="_0603" technology="_4R7" value="4.7k"/>
@@
 <part name="R37" library="daqcs" deviceset="RES" device="_0603" technology="_4R7" value="4.7k"/>
 <part name="C27" library="comms" deviceset="CAP" device="_0603" technology="_100NF0" value="100nF"/>
+<part name="R38" library="comms" deviceset="RES" device="_0805" technology="_0R0" value="0.0"/>
+<part name="R39" library="comms" deviceset="RES" device="_0805" technology="_0R0" value="0.0"/>
+<part name="U9" library="comms" deviceset="UBLOX_MAX" device="" value="MAX-M8Q"/>
 </parts>
 <sheets>
@@
 <instances>
 <instance part="FRAME4" gate="G$1" x="0" y="0"/>
-<instance part="U$1" gate="G$1" x="134.62" y="106.68"/>
 <instance part="R14" gate="G$1" x="50.8" y="101.6" rot="R90"/>
 <instance part="R15" gate="G$1" x="38.1" y="101.6" rot="R90"/>
-<instance part="SUPPLY6" gate="GND" x="104.14" y="68.58"/>
+<instance part="SUPPLY6" gate="GND" x="109.22" y="68.58"/>
 <instance part="J1" gate="G$1" x="55.88" y="116.84"/>
-<instance part="R16" gate="G$1" x="96.52" y="101.6"/>
+<instance part="R16" gate="G$1" x="93.98" y="101.6"/>
 <instance part="C22" gate="G$1" x="76.2" y="78.74"/>
 <instance part="L5" gate="G$1" x="76.2" y="104.14"/>
@@
 <instance part="R18" gate="G$1" x="167.64" y="121.92"/>
 <instance part="C27" gate="G$1" x="220.98" y="109.22"/>
+<instance part="R38" gate="G$1" x="101.6" y="106.68"/>
+<instance part="R39" gate="G$1" x="167.64" y="101.6"/>
+<instance part="U9" gate="G$1" x="134.62" y="106.68"/>
 </instances>
 <busses>
@@
 <net name="3P3V_SENSORS" class="0">
 <segment>
-<pinref part="U$1" gate="G$1" pin="8_VCC"/>
 <wire x1="157.48" y1="116.84" x2="170.18" y2="116.84" width="0.1524" layer="91"/>
-<pinref part="U$1" gate="G$1" pin="7_VCC_IO"/>
 <wire x1="157.48" y1="111.76" x2="170.18" y2="111.76" width="0.1524" layer="91"/>
-<pinref part="U$1" gate="G$1" pin="6_V_BCKP"/>
 <wire x1="157.48" y1="106.68" x2="170.18" y2="106.68" width="0.1524" layer="91"/>
 <wire x1="170.18" y1="106.68" x2="170.18" y2="111.76" width="0.1524" layer="91"/>
@@
 <wire x1="220.98" y1="114.3" x2="220.98" y2="116.84" width="0.1524" layer="91"/>
 <junction x="220.98" y="116.84"/>
+<pinref part="U9" gate="G$1" pin="6_V_BCKP"/>
+<pinref part="U9" gate="G$1" pin="7_VCC_IO"/>
+<pinref part="U9" gate="G$1" pin="8_VCC"/>
 </segment>
 <segment>
@@
 <segment>
 <pinref part="SUPPLY6" gate="GND" pin="GND"/>
-<wire x1="104.14" y1="121.92" x2="104.14" y2="114.3" width="0.1524" layer="91"/>
-<wire x1="104.14" y1="114.3" x2="104.14" y2="111.76" width="0.1524" layer="91"/>
-<wire x1="104.14" y1="111.76" x2="104.14" y2="76.2" width="0.1524" layer="91"/>
-<wire x1="104.14" y1="76.2" x2="104.14" y2="73.66" width="0.1524" layer="91"/>
-<wire x1="104.14" y1="73.66" x2="104.14" y2="71.12" width="0.1524" layer="91"/>
-<pinref part="U$1" gate="G$1" pin="12_GND"/>
-<wire x1="111.76" y1="111.76" x2="104.14" y2="111.76" width="0.1524" layer="91"/>
-<junction x="104.14" y="111.76"/>
+<wire x1="109.22" y1="121.92" x2="109.22" y2="114.3" width="0.1524" layer="91"/>
+<wire x1="109.22" y1="114.3" x2="109.22" y2="111.76" width="0.1524" layer="91"/>
+<wire x1="109.22" y1="111.76" x2="109.22" y2="76.2" width="0.1524" layer="91"/>
+<wire x1="109.22" y1="76.2" x2="109.22" y2="73.66" width="0.1524" layer="91"/>
+<wire x1="109.22" y1="73.66" x2="109.22" y2="71.12" width="0.1524" layer="91"/>
+<wire x1="111.76" y1="111.76" x2="109.22" y2="111.76" width="0.1524" layer="91"/>
+<junction x="109.22" y="111.76"/>
 <wire x1="170.18" y1="81.28" x2="170.18" y2="73.66" width="0.1524" layer="91"/>
-<pinref part="U$1" gate="G$1" pin="1_GND"/>
 <wire x1="157.48" y1="81.28" x2="170.18" y2="81.28" width="0.1524" layer="91"/>
-<wire x1="170.18" y1="73.66" x2="104.14" y2="73.66" width="0.1524" layer="91"/>
-<junction x="104.14" y="73.66"/>
-<pinref part="U$1" gate="G$1" pin="10_GND"/>
-<wire x1="111.76" y1="121.92" x2="104.14" y2="121.92" width="0.1524" layer="91"/>
+<wire x1="170.18" y1="73.66" x2="109.22" y2="73.66" width="0.1524" layer="91"/>
+<junction x="109.22" y="73.66"/>
+<wire x1="111.76" y1="121.92" x2="109.22" y2="121.92" width="0.1524" layer="91"/>
 <pinref part="J1" gate="G$1" pin="GND@1"/>
-<wire x1="58.42" y1="114.3" x2="104.14" y2="114.3" width="0.1524" layer="91"/>
-<junction x="104.14" y="114.3"/>
+<wire x1="58.42" y1="114.3" x2="109.22" y2="114.3" width="0.1524" layer="91"/>
+<junction x="109.22" y="114.3"/>
 <pinref part="C22" gate="G$1" pin="2"/>
-<wire x1="76.2" y1="76.2" x2="104.14" y2="76.2" width="0.1524" layer="91"/>
-<junction x="104.14" y="76.2"/>
+<wire x1="76.2" y1="76.2" x2="109.22" y2="76.2" width="0.1524" layer="91"/>
+<junction x="109.22" y="76.2"/>
 <pinref part="LED1" gate="G$1" pin="C"/>
 <wire x1="198.12" y1="96.52" x2="203.2" y2="96.52" width="0.1524" layer="91"/>
@@
 <wire x1="220.98" y1="73.66" x2="203.2" y2="73.66" width="0.1524" layer="91"/>
 <junction x="203.2" y="73.66"/>
+<pinref part="U9" gate="G$1" pin="1_GND"/>
+<pinref part="U9" gate="G$1" pin="10_GND"/>
+<pinref part="U9" gate="G$1" pin="12_GND"/>
 </segment>
 </net>
@@
 <segment>
 <pinref part="J1" gate="G$1" pin="1"/>
-<pinref part="U$1" gate="G$1" pin="11_RF_IN"/>
 <wire x1="58.42" y1="116.84" x2="76.2" y2="116.84" width="0.1524" layer="91"/>
 <pinref part="L5" gate="G$1" pin="1"/>
@@
 <wire x1="76.2" y1="111.76" x2="76.2" y2="116.84" width="0.1524" layer="91"/>
 <junction x="76.2" y="116.84"/>
+<pinref part="U9" gate="G$1" pin="11_RF_IN"/>
 </segment>
 </net>
@@
 <pinref part="R15" gate="G$1" pin="1"/>
 <wire x1="38.1" y1="96.52" x2="38.1" y2="86.36" width="0.1524" layer="91"/>
-<pinref part="U$1" gate="G$1" pin="17_SCL2"/>
 <wire x1="38.1" y1="86.36" x2="111.76" y2="86.36" width="0.1524" layer="91"/>
 <wire x1="38.1" y1="86.36" x2="10.16" y2="86.36" width="0.1524" layer="91"/>
 <junction x="38.1" y="86.36"/>
 <label x="12.7" y="86.36" size="1.778" layer="95"/>
+<pinref part="U9" gate="G$1" pin="17_SCL2"/>
 </segment>
 </net>
 <net name="GPS_SDA" class="0">
 <segment>
-<pinref part="U$1" gate="G$1" pin="16_SDA2"/>
 <wire x1="111.76" y1="91.44" x2="50.8" y2="91.44" width="0.1524" layer="91"/>
 <pinref part="R14" gate="G$1" pin="1"/>
@@
 <junction x="50.8" y="91.44"/>
 <label x="12.7" y="91.44" size="1.778" layer="95"/>
+<pinref part="U9" gate="G$1" pin="16_SDA2"/>
 </segment>
 </net>
 <net name="N$23" class="0">
 <segment>
-<pinref part="U$1" gate="G$1" pin="4_TIMEPULSE"/>
 <pinref part="R17" gate="G$1" pin="1"/>
 <wire x1="157.48" y1="96.52" x2="172.72" y2="96.52" width="0.1524" layer="91"/>
+<pinref part="U9" gate="G$1" pin="4_TIMEPULSE"/>
 </segment>
 </net>
@@
 <net name="N$26" class="0">
 <segment>
-<pinref part="U$1" gate="G$1" pin="3_RXD1"/>
 <wire x1="157.48" y1="91.44" x2="162.56" y2="91.44" width="0.1524" layer="91"/>
 <pinref part="R19" gate="G$1" pin="1"/>
+<pinref part="U9" gate="G$1" pin="3_RXD1"/>
 </segment>
 </net>
 <net name="N$27" class="0">
 <segment>
-<pinref part="U$1" gate="G$1" pin="2_TXD1"/>
 <wire x1="157.48" y1="86.36" x2="172.72" y2="86.36" width="0.1524" layer="91"/>
 <pinref part="R20" gate="G$1" pin="1"/>
+<pinref part="U9" gate="G$1" pin="2_TXD1"/>
 </segment>
 </net>
 <net name="N$28" class="0">
 <segment>
-<pinref part="U$1" gate="G$1" pin="9_V_RESET"/>
 <wire x1="157.48" y1="121.92" x2="162.56" y2="121.92" width="0.1524" layer="91"/>
 <pinref part="R18" gate="G$1" pin="1"/>
+<pinref part="U9" gate="G$1" pin="9_V_RESET"/>
 </segment>
 </net>
 <net name="N$20" class="0">
 <segment>
-<pinref part="U$1" gate="G$1" pin="14_VCC_RF"/>
 <pinref part="R16" gate="G$1" pin="2"/>
-<wire x1="111.76" y1="101.6" x2="101.6" y2="101.6" width="0.1524" layer="91"/>
+<wire x1="111.76" y1="101.6" x2="99.06" y2="101.6" width="0.1524" layer="91"/>
+<pinref part="U9" gate="G$1" pin="14_VCC_RF"/>
 </segment>
 </net>
@@
 <pinref part="R16" gate="G$1" pin="1"/>
 <wire x1="76.2" y1="93.98" x2="76.2" y2="96.52" width="0.1524" layer="91"/>
-<wire x1="91.44" y1="101.6" x2="86.36" y2="101.6" width="0.1524" layer="91"/>
+<wire x1="88.9" y1="101.6" x2="86.36" y2="101.6" width="0.1524" layer="91"/>
 <wire x1="86.36" y1="101.6" x2="86.36" y2="93.98" width="0.1524" layer="91"/>
 <wire x1="86.36" y1="93.98" x2="76.2" y2="93.98" width="0.1524" layer="91"/>
@@
 </segment>
 </net>
+<net name="N$44" class="0">
+<segment>
+<pinref part="R38" gate="G$1" pin="2"/>
+<wire x1="106.68" y1="106.68" x2="111.76" y2="106.68" width="0.1524" layer="91"/>
+<pinref part="U9" gate="G$1" pin="13_ANTON"/>
+</segment>
+</net>
+<net name="N$45" class="0">
+<segment>
+<pinref part="R39" gate="G$1" pin="1"/>
+<wire x1="157.48" y1="101.6" x2="162.56" y2="101.6" width="0.1524" layer="91"/>
+<pinref part="U9" gate="G$1" pin="5_EXTINT0"/>
+</segment>
+</net>

Commit message: Added digital potentiometer to schematic
Parts:
- removed R36, R37: 4.7k, daqcs:RES_4R7_0603
- added C24, C28: 22uF, comms:CAP_22UF0_1206
- added C25: 100nF, comms:CAP_100NF0_0805
- added C29: 100nF, comms:CAP_100NF0_0603
- added L6: 3.3uH, comms:L_3UH3
- added R40: 33.2k, comms:RES_33R2_0603
- added R41: 10k, comms:RES_10R0_0603
- added U10: (no value), comms:MCP4541-103E/MS
- added U11: TPS562209DDCT, comms:TPS562209DDCR
- R14, R15: value 4.7k -> 0; device daqcs:RES_4R7_0603 -> daqcs:RES_0R0_0603
- renumbered U$2 to J2, U$3 to J3, U$4 to J5, U$5 to J4
Connections:
- net 3P3V_ATV renamed 3P3V_RS232
- removed net GPS_SCL: R15.1, U9.17_SCL2
- removed net GPS_SDA: R14.1, U9.16_SDA2
- removed net PRESS_SCL: U8.SCLK
- removed net PRESS_SDA: R36.1, U8.SDI/SDA
- removed net TEMP_SCL: R32.1, U7.SCL
- removed net TEMP_SDA: R31.1, U7.SDA
- new net 3P3V_DIG_POT: C29.1, L6.2, R40.2, U10.VDD
- new net N$48: R41.2
- new net N$50: R15.2
- new net SCL: R32.1, U7.SCL, U8.SCLK, U9.17_SCL2
- new net SDA: R31.1, U7.SDA, U8.SDI/SDA, U9.16_SDA2
- net 3P3V_SENSORS: no longer R14.2, R15.2, R36.2, R37.2
- net GND: now also C11.2, C12.2, R4.1, U4.GND
- net N$8: now also C25.1; no longer C11.2, C12.2, R4.1, U4.GND
Other:
- note added: "Digital Potentiometer"
