File: eagle/projects/msp430_host_board/page1.sch (EAGLE design)
At the start: 11 parts, among them U1 Value, Y1 32.768kHz, Y2 4MHz

Commit message: Added UART and SPI Molex Connectors to DAQCS Host Board Schematic
Parts:
- added SPI_COMMS_J5: 22-05-7058-05, con-molex:22-05-7058-05
- added UART_1_J1, UART_2_J2, UART_3_J3, UART_4_J4: 22-05-7038-03, con-molex:22-05-7038-03
Connections:
- net COMMS_MISO: now also SPI_COMMS_J5-3.S
- net COMMS_MOSI: now also SPI_COMMS_J5-4.S
- net COMMS_SCLK: now also SPI_COMMS_J5-2.S
- net COMMS_SS: now also SPI_COMMS_J5-1.S
- net GND: now also SPI_COMMS_J5-5.S, UART_1_J1-2.S, UART_2_J2-2.S, UART_3_J3-2.S, UART_4_J4-2.S
- net UART_1_RX: now also UART_1_J1-3.S
- net UART_1_TX: now also UART_1_J1-1.S
- net UART_2_RX: now also UART_2_J2-3.S
- net UART_2_TX: now also UART_2_J2-1.S
- net UART_3_RX: now also UART_3_J3-3.S
- net UART_3_TX: now also UART_3_J3-1.S
- net UART_4_RX: now also UART_4_J4-3.S
- net UART_4_TX: now also UART_4_J4-1.S
Other:
- note added: "Header Connector for SPI COMMS"
- note added: "Header Connector for UART_1"
- note added: "Header Connector for UART_2"
- note added: "Header Connector for UART_3"
- note added: "Header Connector for UART_4"
Changed lines of the file:
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@@
 <setting verticaltext="up"/>
 </settings>
-<grid distance="0.1" unitdist="inch" unit="inch" style="lines" multiple="1" display="no" altdistance="0.01" altunitdist="inch" altunit="inch"/>
+<grid distance="0.1" unitdist="inch" unit="inch" style="lines" multiple="1" display="yes" altdistance="0.01" altunitdist="inch" altunit="inch"/>
 <layers>
 <layer number="1" name="Top" color="4" fill="1" visible="no" active="no"/>
@@
 <part name="Y2" library="SparkFun-FreqCtrl" deviceset="RESONATOR" device="4MHZ" value="4MHz"/>
 <part name="GND3" library="SparkFun-Aesthetics" deviceset="GND" device=""/>
+<part name="FRAME2" library="SparkFun-Aesthetics" deviceset="FRAME-A4L" device=""/>
+<part name="UART_1_J1" library="con-molex" deviceset="22-?-03" device="05-7038"/>
+<part name="UART_2_J2" library="con-molex" deviceset="22-?-03" device="05-7038"/>
+<part name="UART_3_J3" library="con-molex" deviceset="22-?-03" device="05-7038"/>
+<part name="UART_4_J4" library="con-molex" deviceset="22-?-03" device="05-7038"/>
+<part name="SPI_COMMS_J5" library="con-molex" deviceset="22-?-05" device="05-7058"/>
 </parts>
 <sheets>
@@
 </segment>
 </net>
+</nets>
+</sheet>
+<sheet>
+<plain>
+<text x="71.12" y="165.1" size="1.778" layer="91">Header Connector for UART_1</text>
+<text x="127" y="165.1" size="1.778" layer="91">Header Connector for UART_2</text>
+<text x="68.58" y="134.62" size="1.778" layer="91">Header Connector for UART_3</text>
+<text x="127" y="134.62" size="1.778" layer="91">Header Connector for UART_4</text>
+<text x="68.58" y="104.14" size="1.778" layer="91">Header Connector for SPI COMMS</text>
+</plain>
+<instances>
+<instance part="FRAME2" gate="G$1" x="40.64" y="2.54"/>
+<instance part="UART_1_J1" gate="-1" x="91.44" y="157.48"/>
+<instance part="UART_1_J1" gate="-2" x="91.44" y="152.4"/>
+<instance part="UART_1_J1" gate="-3" x="91.44" y="147.32"/>
+<instance part="UART_2_J2" gate="-1" x="147.32" y="157.48"/>
+<instance part="UART_2_J2" gate="-2" x="147.32" y="152.4"/>
+<instance part="UART_2_J2" gate="-3" x="147.32" y="147.32"/>
+<instance part="UART_3_J3" gate="-1" x="88.9" y="127"/>
+<instance part="UART_3_J3" gate="-2" x="88.9" y="121.92"/>
+<instance part="UART_3_J3" gate="-3" x="88.9" y="116.84"/>
+<instance part="UART_4_J4" gate="-1" x="147.32" y="127"/>
+<instance part="UART_4_J4" gate="-2" x="147.32" y="121.92"/>
+<instance part="UART_4_J4" gate="-3" x="147.32" y="116.84"/>
+<instance part="SPI_COMMS_J5" gate="-1" x="88.9" y="96.52"/>
+<instance part="SPI_COMMS_J5" gate="-2" x="88.9" y="91.44"/>
+<instance part="SPI_COMMS_J5" gate="-3" x="88.9" y="86.36"/>
+<instance part="SPI_COMMS_J5" gate="-4" x="88.9" y="81.28"/>
+<instance part="SPI_COMMS_J5" gate="-5" x="88.9" y="76.2"/>
+</instances>
+<busses>
+</busses>
+<nets>
+<net name="UART_1_TX" class="0">
+<segment>
+<pinref part="UART_1_J1" gate="-1" pin="S"/>
+<wire x1="88.9" y1="157.48" x2="68.58" y2="157.48" width="0.1524" layer="91"/>
+<label x="68.58" y="157.48" size="1.778" layer="95"/>
+</segment>
+</net>
+<net name="GND" class="0">
+<segment>
+<pinref part="UART_1_J1" gate="-2" pin="S"/>
+<wire x1="88.9" y1="152.4" x2="68.58" y2="152.4" width="0.1524" layer="91"/>
+<label x="68.58" y="152.4" size="1.778" layer="95"/>
+</segment>
+<segment>
+<pinref part="UART_2_J2" gate="-2" pin="S"/>
+<wire x1="144.78" y1="152.4" x2="124.46" y2="152.4" width="0.1524" layer="91"/>
+<label x="124.46" y="152.4" size="1.778" layer="95"/>
+</segment>
+<segment>
+<pinref part="UART_3_J3" gate="-2" pin="S"/>
+<wire x1="86.36" y1="121.92" x2="66.04" y2="121.92" width="0.1524" layer="91"/>
+<label x="66.04" y="121.92" size="1.778" layer="95"/>
+</segment>
+<segment>
+<pinref part="UART_4_J4" gate="-2" pin="S"/>
+<wire x1="144.78" y1="121.92" x2="124.46" y2="121.92" width="0.1524" layer="91"/>
+<label x="124.46" y="121.92" size="1.778" layer="95"/>
+</segment>
+<segment>
+<pinref part="SPI_COMMS_J5" gate="-5" pin="S"/>
+<wire x1="86.36" y1="76.2" x2="66.04" y2="76.2" width="0.1524" layer="91"/>
+<label x="66.04" y="76.2" size="1.778" layer="95"/>
+</segment>
+</net>
+<net name="UART_1_RX" class="0">
+<segment>
+<pinref part="UART_1_J1" gate="-3" pin="S"/>
+<wire x1="88.9" y1="147.32" x2="68.58" y2="147.32" width="0.1524" layer="91"/>
+<label x="68.58" y="147.32" size="1.778" layer="95"/>
+</segment>
+</net>
+<net name="UART_2_TX" class="0">
+<segment>
+<pinref part="UART_2_J2" gate="-1" pin="S"/>
+<wire x1="144.78" y1="157.48" x2="124.46" y2="157.48" width="0.1524" layer="91"/>
+<label x="124.46" y="157.48" size="1.778" layer="95"/>
+</segment>
+</net>
+<net name="UART_2_RX" class="0">
+<segment>
+<pinref part="UART_2_J2" gate="-3" pin="S"/>
+<wire x1="144.78" y1="147.32" x2="124.46" y2="147.32" width="0.1524" layer="91"/>
+<label x="124.46" y="147.32" size="1.778" layer="95"/>
+</segment>
+</net>
+<net name="UART_3_RX" class="0">
+<segment>
+<pinref part="UART_3_J3" gate="-3" pin="S"/>
+<wire x1="86.36" y1="116.84" x2="66.04" y2="116.84" width="0.1524" layer="91"/>
+<label x="66.04" y="116.84" size="1.778" layer="95"/>
+</segment>
+</net>
+<net name="UART_4_TX" class="0">
+<segment>
+<pinref part="UART_4_J4" gate="-1" pin="S"/>
+<wire x1="144.78" y1="127" x2="124.46" y2="127" width="0.1524" layer="91"/>
+<label x="124.46" y="127" size="1.778" layer="95"/>
+</segment>
+</net>
+<net name="UART_4_RX" class="0">
+<segment>
+<pinref part="UART_4_J4" gate="-3" pin="S"/>
+<wire x1="144.78" y1="116.84" x2="124.46" y2="116.84" width="0.1524" layer="91"/>
+<label x="124.46" y="116.84" size="1.778" layer="95"/>
+</segment>
+</net>
+<net name="UART_3_TX" class="0">
+<segment>
+<pinref part="UART_3_J3" gate="-1" pin="S"/>
+<wire x1="86.36" y1="127" x2="66.04" y2="127" width="0.1524" layer="91"/>
+<label x="66.04" y="127" size="1.778" layer="95"/>
+</segment>
+</net>
+<net name="N$5" class="0">
+<segment>
+<wire x1="60.96" y1="165.1" x2="111.76" y2="165.1" width="0.1524" layer="91"/>
+<wire x1="111.76" y1="165.1" x2="111.76" y2="142.24" width="0.1524" layer="91"/>
+<wire x1="111.76" y1="142.24" x2="60.96" y2="142.24" width="0.1524" layer="91"/>
+<wire x1="60.96" y1="142.24" x2="60.96" y2="165.1" width="0.1524" layer="91"/>
+</segment>
+</net>
+<net name="N$6" class="0">
+<segment>
+<wire x1="119.38" y1="165.1" x2="167.64" y2="165.1" width="0.1524" layer="91"/>
+<wire x1="167.64" y1="165.1" x2="167.64" y2="142.24" width="0.1524" layer="91"/>
+<wire x1="167.64" y1="142.24" x2="119.38" y2="142.24" width="0.1524" layer="91"/>
+<wire x1="119.38" y1="142.24" x2="119.38" y2="165.1" width="0.1524" layer="91"/>
+</segment>
+</net>
+<net name="N$7" class="0">
+<segment>
+<wire x1="60.96" y1="134.62" x2="111.76" y2="134.62" width="0.1524" layer="91"/>
+<wire x1="111.76" y1="134.62" x2="111.76" y2="111.76" width="0.1524" layer="91"/>
+<wire x1="111.76" y1="111.76" x2="60.96" y2="111.76" width="0.1524" layer="91"/>
+<wire x1="60.96" y1="111.76" x2="60.96" y2="134.62" width="0.1524" layer="91"/>
+</segment>
+</net>
+<net name="N$8" class="0">
+<segment>
+<wire x1="119.38" y1="134.62" x2="167.64" y2="134.62" width="0.1524" layer="91"/>
+<wire x1="167.64" y1="134.62" x2="167.64" y2="111.76" width="0.1524" layer="91"/>
+<wire x1="167.64" y1="111.76" x2="119.38" y2="111.76" width="0.1524" layer="91"/>
+<wire x1="119.38" y1="111.76" x2="119.38" y2="134.62" width="0.1524" layer="91"/>
+</segment>
+</net>
+<net name="COMMS_SS" class="0">
+<segment>
+<pinref part="SPI_COMMS_J5" gate="-1" pin="S"/>
+<wire x1="86.36" y1="96.52" x2="66.04" y2="96.52" width="0.1524" layer="91"/>
+<label x="66.04" y="96.52" size="1.778" layer="95"/>
+</segment>
+</net>
+<net name="COMMS_SCLK" class="0">
+<segment>
+<pinref part="SPI_COMMS_J5" gate="-2" pin="S"/>
+<wire x1="86.36" y1="91.44" x2="66.04" y2="91.44" width="0.1524" layer="91"/>
+<label x="66.04" y="91.44" size="1.778" layer="95"/>
+</segment>
+</net>
+<net name="COMMS_MISO" class="0">
+<segment>
+<pinref part="SPI_COMMS_J5" gate="-3" pin="S"/>
+<wire x1="86.36" y1="86.36" x2="66.04" y2="86.36" width="0.1524" layer="91"/>
+<label x="66.04" y="86.36" size="1.778" layer="95"/>
+</segment>
+</net>
+<net name="COMMS_MOSI" class="0">
+<segment>
+<pinref part="SPI_COMMS_J5" gate="-4" pin="S"/>
+<wire x1="86.36" y1="81.28" x2="66.04" y2="81.28" width="0.1524" layer="91"/>
+<label x="66.04" y="81.28" size="1.778" layer="95"/>
+</segment>
+</net>
+<net name="N$9" class="0">
+<segment>
+<wire x1="60.96" y1="104.14" x2="111.76" y2="104.14" width="0.1524" layer="91"/>
+<wire x1="111.76" y1="104.14" x2="111.76" y2="71.12" width="0.1524" layer="91"/>
+<wire x1="111.76" y1="71.12" x2="60.96" y2="71.12" width="0.1524" layer="91"/>
+<wire x1="60.96" y1="71.12" x2="60.96" y2="104.14" width="0.1524" layer="91"/>
+</segment>
+</net>

Commit message: Added JTAG header
Parts:
- added JTAG_J6: (no value), SparkFun-Connectors:M02PTH
Connections:
- new net SBWTCK: JTAG_J6.1, U1.TEST_SBWTCK
- new net SBWTDIO: JTAG_J6.2, U1.RST_NMI_SBWTDIO_N
Other:
- note added: "Header Connector for JTAG"
Changed lines of the file:
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@@
 <layer number="112" name="tSilk" color="7" fill="1" visible="yes" active="yes"/>
 <layer number="113" name="ReferenceLS" color="7" fill="1" visible="no" active="no"/>
+<layer number="114" name="Badge_Outline" color="7" fill="1" visible="yes" active="yes"/>
+<layer number="115" name="ReferenceISLANDS" color="7" fill="1" visible="yes" active="yes"/>
 <layer number="116" name="Patch_BOT" color="9" fill="4" visible="yes" active="yes"/>
 <layer number="118" name="Rect_Pads" color="7" fill="1" visible="no" active="no"/>
@@
 <parts>
 <part name="U1" library="daqcs_host" deviceset="MSP430FR5994IPNR" device="" value="Value"/>
-<part name="FRAME1" library="SparkFun-Aesthetics" deviceset="FRAME-A4L" device=""/>
 <part name="3V3" library="SparkFun-Aesthetics" deviceset="3.3V" device="" value="+3.3V"/>
 <part name="SUPPLY2" library="SparkFun-Aesthetics" deviceset="3.3V" device="" value="+3.3V"/>
@@
 <part name="Y2" library="SparkFun-FreqCtrl" deviceset="RESONATOR" device="4MHZ" value="4MHz"/>
 <part name="GND3" library="SparkFun-Aesthetics" deviceset="GND" device=""/>
-<part name="FRAME2" library="SparkFun-Aesthetics" deviceset="FRAME-A4L" device=""/>
 <part name="UART_1_J1" library="con-molex" deviceset="22-?-03" device="05-7038"/>
 <part name="UART_2_J2" library="con-molex" deviceset="22-?-03" device="05-7038"/>
@@
 <part name="UART_4_J4" library="con-molex" deviceset="22-?-03" device="05-7038"/>
 <part name="SPI_COMMS_J5" library="con-molex" deviceset="22-?-05" device="05-7058"/>
+<part name="FRAME1" library="frames" deviceset="A3L-LOC" device=""/>
+<part name="FRAME2" library="frames" deviceset="A3L-LOC" device=""/>
+<part name="JTAG_J6" library="SparkFun-Connectors" deviceset="M02" device="PTH"/>
 </parts>
 <sheets>
@@
 <attribute name="PARTNUMBER" x="43.18" y="48.26" size="1.778" layer="96" display="off"/>
 </instance>
-<instance part="FRAME1" gate="G$1" x="-78.74" y="-55.88"/>
 <instance part="3V3" gate="G$1" x="-71.12" y="114.3"/>
 <instance part="SUPPLY2" gate="G$1" x="180.34" y="5.08"/>
@@
 <instance part="Y2" gate="G$1" x="-45.72" y="-35.56"/>
 <instance part="GND3" gate="1" x="-45.72" y="-48.26"/>
+<instance part="FRAME1" gate="G$1" x="-144.78" y="-93.98"/>
 </instances>
 <busses>
@@
 </segment>
 </net>
+<net name="SBWTCK" class="0">
+<segment>
+<pinref part="U1" gate="A" pin="TEST_SBWTCK"/>
+<wire x1="129.54" y1="25.4" x2="147.32" y2="25.4" width="0.1524" layer="91"/>
+<label x="139.7" y="25.4" size="1.778" layer="95"/>
+</segment>
+</net>
+<net name="SBWTDIO" class="0">
+<segment>
+<pinref part="U1" gate="A" pin="RST_NMI_SBWTDIO_N"/>
+<wire x1="129.54" y1="17.78" x2="147.32" y2="17.78" width="0.1524" layer="91"/>
+<label x="139.7" y="17.78" size="1.778" layer="95"/>
+</segment>
+</net>
 </nets>
 </sheet>
@@
 <text x="127" y="134.62" size="1.778" layer="91">Header Connector for UART_4</text>
 <text x="68.58" y="104.14" size="1.778" layer="91">Header Connector for SPI COMMS</text>
+<text x="213.36" y="165.1" size="1.778" layer="91">Header Connector for JTAG</text>
 </plain>
 <instances>
-<instance part="FRAME2" gate="G$1" x="40.64" y="2.54"/>
 <instance part="UART_1_J1" gate="-1" x="91.44" y="157.48"/>
 <instance part="UART_1_J1" gate="-2" x="91.44" y="152.4"/>
@@
 <instance part="SPI_COMMS_J5" gate="-4" x="88.9" y="81.28"/>
 <instance part="SPI_COMMS_J5" gate="-5" x="88.9" y="76.2"/>
+<instance part="FRAME2" gate="G$1" x="15.24" y="-53.34"/>
+<instance part="JTAG_J6" gate="G$1" x="215.9" y="152.4"/>
 </instances>
 <busses>
@@
 </segment>
 </net>
+<net name="SBWTDIO" class="0">
+<segment>
+<pinref part="JTAG_J6" gate="G$1" pin="2"/>
+<wire x1="223.52" y1="154.94" x2="243.84" y2="154.94" width="0.1524" layer="91"/>
+<label x="236.22" y="154.94" size="1.778" layer="95"/>
+</segment>
+</net>
+<net name="SBWTCK" class="0">
+<segment>
+<pinref part="JTAG_J6" gate="G$1" pin="1"/>
+<wire x1="223.52" y1="152.4" x2="243.84" y2="152.4" width="0.1524" layer="91"/>
+<label x="236.22" y="152.4" size="1.778" layer="95"/>
+</segment>
+</net>
+<net name="N$10" class="0">
+<segment>
+<wire x1="200.66" y1="165.1" x2="254" y2="165.1" width="0.1524" layer="91"/>
+<wire x1="254" y1="165.1" x2="254" y2="142.24" width="0.1524" layer="91"/>
+<wire x1="254" y1="142.24" x2="200.66" y2="142.24" width="0.1524" layer="91"/>
+<wire x1="200.66" y1="142.24" x2="200.66" y2="165.1" width="0.1524" layer="91"/>
+</segment>
+</net>

Commit message: Added Reset Push Button, new 47k res, 1000pF cap
Parts:
- added C8: 1000pF, daqcs_host:CAP_1000PF0_0603
- added R2: 47k, daqcs_host:RES_47R0_0603
- added S1: SWITCH-MOMENTARY-2PTH, SparkFun-Electromechanical:SWITCH-MOMENTARY-2PTH
Connections:
- removed net SBWTDIO: JTAG_J6.2, U1.RST_NMI_SBWTDIO_N
- new net RST_SBWTDIO: C8.1, JTAG_J6.2, R2.2, S1.2, U1.RST_NMI_SBWTDIO_N
- net 3V3: now also R2.1
- net GND: now also C8.2, S1.1
Other:
- note added: "Reset Pushbutton"
Changed lines of the file:
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@@
 <setting verticaltext="up"/>
 </settings>
-<grid distance="0.1" unitdist="inch" unit="inch" style="lines" multiple="1" display="yes" altdistance="0.01" altunitdist="inch" altunit="inch"/>
+<grid distance="0.1" unitdist="inch" unit="inch" style="lines" multiple="1" display="no" altdistance="0.01" altunitdist="inch" altunit="inch"/>
 <layers>
 <layer number="1" name="Top" color="4" fill="1" visible="no" active="no"/>
@@
 <part name="FRAME2" library="frames" deviceset="A3L-LOC" device=""/>
 <part name="JTAG_J6" library="SparkFun-Connectors" deviceset="M02" device="PTH"/>
+<part name="S1" library="SparkFun-Electromechanical" deviceset="SWITCH-MOMENTARY-2" device="PTH"/>
+<part name="R2" library="daqcs_host" deviceset="RES" device="_0603" technology="_47R0" value="47k"/>
+<part name="C8" library="daqcs_host" deviceset="CAP" device="_0603" technology="_1000PF0" value="1000pF"/>
+<part name="GND4" library="SparkFun-Aesthetics" deviceset="GND" device=""/>
+<part name="GND5" library="SparkFun-Aesthetics" deviceset="GND" device=""/>
+<part name="SUPPLY1" library="SparkFun-Aesthetics" deviceset="3.3V" device="" value="3.3V"/>
 </parts>
 <sheets>
@@
 <wire x1="160.02" y1="-7.62" x2="160.02" y2="-5.08" width="0.1524" layer="91"/>
 <junction x="160.02" y="-5.08"/>
+<label x="182.88" y="0" size="1.778" layer="95"/>
 </segment>
 </net>
@@
 </segment>
 </net>
-<net name="SBWTDIO" class="0">
+<net name="RST_SBWTDIO" class="0">
 <segment>
 <pinref part="U1" gate="A" pin="RST_NMI_SBWTDIO_N"/>
@@
 <text x="68.58" y="104.14" size="1.778" layer="91">Header Connector for SPI COMMS</text>
 <text x="213.36" y="165.1" size="1.778" layer="91">Header Connector for JTAG</text>
+<text x="322.58" y="165.1" size="1.778" layer="91">Reset Pushbutton</text>
 </plain>
 <instances>
@@
 <instance part="FRAME2" gate="G$1" x="15.24" y="-53.34"/>
 <instance part="JTAG_J6" gate="G$1" x="215.9" y="152.4"/>
+<instance part="S1" gate="G$1" x="304.8" y="139.7"/>
+<instance part="R2" gate="G$1" x="337.82" y="149.86" smashed="yes" rot="R270">
+<attribute name="NAME" x="341.8586" y="148.59" size="1.778" layer="95"/>
+<attribute name="VALUE" x="331.978" y="148.59" size="1.778" layer="96"/>
+</instance>
+<instance part="C8" gate="G$1" x="337.82" y="129.54"/>
+<instance part="GND4" gate="1" x="294.64" y="129.54"/>
+<instance part="GND5" gate="1" x="337.82" y="119.38"/>
+<instance part="SUPPLY1" gate="G$1" x="337.82" y="157.48"/>
 </instances>
 <busses>
@@
 <label x="66.04" y="76.2" size="1.778" layer="95"/>
 </segment>
+<segment>
+<pinref part="GND4" gate="1" pin="GND"/>
+<wire x1="294.64" y1="132.08" x2="294.64" y2="139.7" width="0.1524" layer="91"/>
+<pinref part="S1" gate="G$1" pin="1"/>
+<wire x1="294.64" y1="139.7" x2="299.72" y2="139.7" width="0.1524" layer="91"/>
+</segment>
+<segment>
+<pinref part="C8" gate="G$1" pin="2"/>
+<pinref part="GND5" gate="1" pin="GND"/>
+<wire x1="337.82" y1="127" x2="337.82" y2="121.92" width="0.1524" layer="91"/>
+</segment>
 </net>
 <net name="UART_1_RX" class="0">
@@
 </segment>
 </net>
-<net name="SBWTDIO" class="0">
+<net name="RST_SBWTDIO" class="0">
 <segment>
 <pinref part="JTAG_J6" gate="G$1" pin="2"/>
 <wire x1="223.52" y1="154.94" x2="243.84" y2="154.94" width="0.1524" layer="91"/>
 <label x="236.22" y="154.94" size="1.778" layer="95"/>
+</segment>
+<segment>
+<pinref part="S1" gate="G$1" pin="2"/>
+<pinref part="R2" gate="G$1" pin="2"/>
+<wire x1="309.88" y1="139.7" x2="337.82" y2="139.7" width="0.1524" layer="91"/>
+<wire x1="337.82" y1="139.7" x2="337.82" y2="144.78" width="0.1524" layer="91"/>
+<pinref part="C8" gate="G$1" pin="1"/>
+<wire x1="337.82" y1="139.7" x2="337.82" y2="134.62" width="0.1524" layer="91"/>
+<junction x="337.82" y="139.7"/>
+<wire x1="337.82" y1="139.7" x2="358.14" y2="139.7" width="0.1524" layer="91"/>
+<label x="355.6" y="139.7" size="1.778" layer="95"/>
 </segment>
 </net>
@@
 </segment>
 </net>
+<net name="3V3" class="0">
+<segment>
+<pinref part="R2" gate="G$1" pin="1"/>
+<pinref part="SUPPLY1" gate="G$1" pin="3.3V"/>
+<wire x1="337.82" y1="154.94" x2="337.82" y2="157.48" width="0.1524" layer="91"/>
+<label x="340.36" y="154.94" size="1.778" layer="95"/>
+</segment>
+</net>
+<net name="N$11" class="0">
+<segment>
+<wire x1="281.94" y1="165.1" x2="381" y2="165.1" width="0.1524" layer="91"/>
+<wire x1="381" y1="165.1" x2="381" y2="111.76" width="0.1524" layer="91"/>
+<wire x1="381" y1="111.76" x2="281.94" y2="111.76" width="0.1524" layer="91"/>
+<wire x1="281.94" y1="111.76" x2="281.94" y2="165.1" width="0.1524" layer="91"/>
+</segment>
+</net>

Commit message: Added connectors for motor controller
Parts:
- added MOTOR_AN_IN_J8: 22-05-7038-03, con-molex:22-05-7038-03
- added MOTOR_DIG_OUT_J7: 22-05-7058-05, con-molex:22-05-7058-05
Connections:
- net ACT_CURRENT_IN: now also MOTOR_AN_IN_J8-2.S
- net ACT_SPEED_IN: now also MOTOR_AN_IN_J8-1.S
- net CURRENT_PWM_OUT: now also MOTOR_DIG_OUT_J7-2.S
- net DIR_MOTOR_OUT: now also MOTOR_DIG_OUT_J7-4.S
- net EN_MOTOR_OUT: now also MOTOR_DIG_OUT_J7-3.S
- net GND: now also MOTOR_AN_IN_J8-3.S, MOTOR_DIG_OUT_J7-5.S
- net SPEED_PWM_OUT: now also MOTOR_DIG_OUT_J7-1.S
Other:
- note added: "Header Connector for Motor In"
- note added: "Header Connector for Motor Out"
- moved on the sheet: UART_2_J2-1, UART_2_J2-2, UART_2_J2-3, UART_4_J4-1, UART_4_J4-2, UART_4_J4-3

Commit message: Swapped 3 pin Uart connector with 4 pin to add RST signal
Parts:
- UART_1_J1, UART_2_J2, UART_3_J3, UART_4_J4: value 22-05-7038-03 -> 22-05-7048-04; device con-molex:22-05-7038-03 -> con-molex:22-05-7048-04
Connections:
- new net RST_PI_1: U1.P4.4_TB0.5, UART_1_J1-4.S
- new net RST_PI_2: U1.P4.5, UART_2_J2-4.S
- new net RST_PI_3: U1.P4.6, UART_3_J3-4.S
- new net RST_PI_4: U1.P4.7, UART_4_J4-4.S
Other:
- moved on the sheet: UART_1_J1-1, UART_1_J1-2, UART_1_J1-3, UART_2_J2-1, UART_2_J2-2, UART_2_J2-3, UART_3_J3-1, UART_3_J3-2, UART_3_J3-3, UART_4_J4-1, UART_4_J4-2, UART_4_J4-3
