File: eagle/projects/msp430_host_board/page1.sch (EAGLE design)
At the start: 22 parts, among them U1 Value, Y1 32.768kHz, Y2 4MHz

Commit message: Added pressure and temperature sensors. New 2.61k RES in library
Parts:
- added C10, C9: 100nF, daqcs_host:CAP_100NF0_0603
- added R3, R4: 2.61k, daqcs_host:RES_2R61_0603
- added U2: PCT2075D,118, daqcs_host:PCT2075D,118SOIC8
- added U3: MS560702BA03-50, daqcs_host:MS5607-02BA03_8SMD
Connections:
- new net SENSE_SCL: R4.2, U1.P6.5_UCB3SOMI_UCB3SCL, U2.SCL, U3.SCLK
- new net SENSE_SDA: R3.2, U1.P6.4_UCB3SIMO_UCB3SDA, U2.SDA, U3.SDI/SDA
- net 3V3: now also C10.1, C9.1, R3.1, R4.1, U2.VCC, U3.PS, U3.VDD
- net GND: now also C10.2, C9.2, U2.A0, U2.A1, U2.A2, U2.GND, U3.CSB@1, U3.CSB@2, U3.GND
Other:
- note added: "Need to Confirm Proper Pullup RES values"
Changed lines of the file:
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@@
 <part name="UART_3_J3" library="con-molex" deviceset="22-?-04" device="05-7048"/>
 <part name="UART_4_J4" library="con-molex" deviceset="22-?-04" device="05-7048"/>
+<part name="FRAME3" library="frames" deviceset="A3L-LOC" device=""/>
+<part name="U2" library="daqcs_host" deviceset="PCT2075" device="SOIC8" technology="D,118" value="PCT2075D,118"/>
+<part name="SUPPLY3" library="SparkFun-Aesthetics" deviceset="3.3V" device=""/>
+<part name="GND6" library="SparkFun-Aesthetics" deviceset="GND" device=""/>
+<part name="GND7" library="SparkFun-Aesthetics" deviceset="GND" device=""/>
+<part name="U3" library="daqcs_host" deviceset="MS5607" device="_8SMD" technology="-02BA03" value="MS560702BA03-50"/>
+<part name="SUPPLY4" library="SparkFun-Aesthetics" deviceset="3.3V" device=""/>
+<part name="GND8" library="SparkFun-Aesthetics" deviceset="GND" device=""/>
+<part name="GND9" library="SparkFun-Aesthetics" deviceset="GND" device=""/>
+<part name="C9" library="daqcs_host" deviceset="CAP" device="_0603" technology="_100NF0" value="100nF"/>
+<part name="C10" library="daqcs_host" deviceset="CAP" device="_0603" technology="_100NF0" value="100nF"/>
+<part name="R3" library="daqcs_host" deviceset="RES" device="_0603" technology="_2R61" value="2.61k"/>
+<part name="R4" library="daqcs_host" deviceset="RES" device="_0603" technology="_2R61" value="2.61k"/>
+<part name="SUPPLY5" library="SparkFun-Aesthetics" deviceset="3.3V" device=""/>
 </parts>
 <sheets>
 <sheet>
 <plain>
+<text x="193.04" y="68.58" size="1.778" layer="91">Need to Confirm Proper Pullup RES values</text>
 </plain>
 <instances>
@@
 <instance part="GND3" gate="1" x="-45.72" y="-48.26"/>
 <instance part="FRAME1" gate="G$1" x="-144.78" y="-93.98"/>
+<instance part="R3" gate="G$1" x="180.34" y="63.5" smashed="yes" rot="R270">
+<attribute name="NAME" x="181.8386" y="64.77" size="1.778" layer="95"/>
+<attribute name="VALUE" x="182.118" y="62.23" size="1.778" layer="96"/>
+</instance>
+<instance part="R4" gate="G$1" x="193.04" y="63.5" smashed="yes" rot="R270">
+<attribute name="NAME" x="194.5386" y="64.77" size="1.778" layer="95"/>
+<attribute name="VALUE" x="194.818" y="62.23" size="1.778" layer="96"/>
+</instance>
+<instance part="SUPPLY5" gate="G$1" x="185.42" y="76.2"/>
 </instances>
 <busses>
@@
 <junction x="160.02" y="-5.08"/>
 <label x="182.88" y="0" size="1.778" layer="95"/>
+</segment>
+<segment>
+<pinref part="R3" gate="G$1" pin="1"/>
+<wire x1="180.34" y1="68.58" x2="180.34" y2="73.66" width="0.1524" layer="91"/>
+<pinref part="R4" gate="G$1" pin="1"/>
+<wire x1="180.34" y1="73.66" x2="185.42" y2="73.66" width="0.1524" layer="91"/>
+<wire x1="185.42" y1="73.66" x2="193.04" y2="73.66" width="0.1524" layer="91"/>
+<wire x1="193.04" y1="73.66" x2="193.04" y2="68.58" width="0.1524" layer="91"/>
+<pinref part="SUPPLY5" gate="G$1" pin="3.3V"/>
+<wire x1="185.42" y1="76.2" x2="185.42" y2="73.66" width="0.1524" layer="91"/>
+<junction x="185.42" y="73.66"/>
+<label x="187.96" y="73.66" size="1.778" layer="95"/>
 </segment>
 </net>
@@
 <wire x1="129.54" y1="71.12" x2="147.32" y2="71.12" width="0.1524" layer="91"/>
 <label x="139.7" y="71.12" size="1.778" layer="95"/>
+</segment>
+</net>
+<net name="SENSE_SDA" class="0">
+<segment>
+<pinref part="U1" gate="A" pin="P6.4_UCB3SIMO_UCB3SDA"/>
+<label x="139.7" y="55.88" size="1.778" layer="95"/>
+<pinref part="R3" gate="G$1" pin="2"/>
+<wire x1="129.54" y1="55.88" x2="180.34" y2="55.88" width="0.1524" layer="91"/>
+<wire x1="180.34" y1="55.88" x2="180.34" y2="58.42" width="0.1524" layer="91"/>
+</segment>
+</net>
+<net name="SENSE_SCL" class="0">
+<segment>
+<pinref part="U1" gate="A" pin="P6.5_UCB3SOMI_UCB3SCL"/>
+<label x="139.7" y="53.34" size="1.778" layer="95"/>
+<pinref part="R4" gate="G$1" pin="2"/>
+<wire x1="129.54" y1="53.34" x2="193.04" y2="53.34" width="0.1524" layer="91"/>
+<wire x1="193.04" y1="53.34" x2="193.04" y2="58.42" width="0.1524" layer="91"/>
 </segment>
 </net>
@@
 </segment>
 </net>
+</nets>
+</sheet>
+<sheet>
+<plain>
+</plain>
+<instances>
+<instance part="FRAME3" gate="G$1" x="-38.1" y="-12.7"/>
+<instance part="U2" gate="A" x="58.42" y="162.56"/>
+<instance part="SUPPLY3" gate="G$1" x="15.24" y="177.8"/>
+<instance part="GND6" gate="1" x="30.48" y="139.7"/>
+<instance part="GND7" gate="1" x="83.82" y="139.7"/>
+<instance part="U3" gate="G$1" x="226.06" y="162.56"/>
+<instance part="SUPPLY4" gate="G$1" x="180.34" y="180.34"/>
+<instance part="GND8" gate="1" x="251.46" y="137.16"/>
+<instance part="GND9" gate="1" x="180.34" y="129.54"/>
+<instance part="C9" gate="G$1" x="180.34" y="142.24"/>
+<instance part="C10" gate="G$1" x="15.24" y="157.48"/>
+</instances>
+<busses>
+</busses>
+<nets>
+<net name="3V3" class="0">
+<segment>
+<pinref part="SUPPLY3" gate="G$1" pin="3.3V"/>
+<wire x1="15.24" y1="177.8" x2="15.24" y2="170.18" width="0.1524" layer="91"/>
+<pinref part="U2" gate="A" pin="VCC"/>
+<wire x1="15.24" y1="170.18" x2="40.64" y2="170.18" width="0.1524" layer="91"/>
+<label x="17.78" y="170.18" size="1.778" layer="95"/>
+<pinref part="C10" gate="G$1" pin="1"/>
+<wire x1="15.24" y1="170.18" x2="15.24" y2="162.56" width="0.1524" layer="91"/>
+<junction x="15.24" y="170.18"/>
+</segment>
+<segment>
+<pinref part="SUPPLY4" gate="G$1" pin="3.3V"/>
+<wire x1="180.34" y1="180.34" x2="180.34" y2="170.18" width="0.1524" layer="91"/>
+<pinref part="U3" gate="G$1" pin="VDD"/>
+<wire x1="180.34" y1="170.18" x2="208.28" y2="170.18" width="0.1524" layer="91"/>
+<label x="185.42" y="170.18" size="1.778" layer="95"/>
+<pinref part="U3" gate="G$1" pin="PS"/>
+<wire x1="208.28" y1="149.86" x2="180.34" y2="149.86" width="0.1524" layer="91"/>
+<wire x1="180.34" y1="149.86" x2="180.34" y2="170.18" width="0.1524" layer="91"/>
+<junction x="180.34" y="170.18"/>
+<pinref part="C9" gate="G$1" pin="1"/>
+<wire x1="180.34" y1="149.86" x2="180.34" y2="147.32" width="0.1524" layer="91"/>
+<junction x="180.34" y="149.86"/>
+</segment>
+</net>
+<net name="GND" class="0">
+<segment>
+<pinref part="U2" gate="A" pin="A0"/>
+<pinref part="GND6" gate="1" pin="GND"/>
+<wire x1="40.64" y1="160.02" x2="30.48" y2="160.02" width="0.1524" layer="91"/>
+<wire x1="30.48" y1="160.02" x2="30.48" y2="154.94" width="0.1524" layer="91"/>
+<pinref part="U2" gate="A" pin="A1"/>
+<wire x1="30.48" y1="154.94" x2="30.48" y2="149.86" width="0.1524" layer="91"/>
+<wire x1="30.48" y1="149.86" x2="30.48" y2="142.24" width="0.1524" layer="91"/>
+<wire x1="40.64" y1="154.94" x2="30.48" y2="154.94" width="0.1524" layer="91"/>
+<junction x="30.48" y="154.94"/>
+<pinref part="U2" gate="A" pin="A2"/>
+<wire x1="40.64" y1="149.86" x2="30.48" y2="149.86" width="0.1524" layer="91"/>
+<junction x="30.48" y="149.86"/>
+<pinref part="C10" gate="G$1" pin="2"/>
+<wire x1="15.24" y1="154.94" x2="15.24" y2="149.86" width="0.1524" layer="91"/>
+<wire x1="15.24" y1="149.86" x2="30.48" y2="149.86" width="0.1524" layer="91"/>
+</segment>
+<segment>
+<pinref part="U2" gate="A" pin="GND"/>
+<pinref part="GND7" gate="1" pin="GND"/>
+<wire x1="76.2" y1="149.86" x2="83.82" y2="149.86" width="0.1524" layer="91"/>
+<wire x1="83.82" y1="149.86" x2="83.82" y2="142.24" width="0.1524" layer="91"/>
+</segment>
+<segment>
+<pinref part="U3" gate="G$1" pin="GND"/>
+<pinref part="GND8" gate="1" pin="GND"/>
+<wire x1="243.84" y1="149.86" x2="251.46" y2="149.86" width="0.1524" layer="91"/>
+<wire x1="251.46" y1="149.86" x2="251.46" y2="139.7" width="0.1524" layer="91"/>
+</segment>
+<segment>
+<pinref part="GND9" gate="1" pin="GND"/>
+<wire x1="180.34" y1="132.08" x2="180.34" y2="137.16" width="0.1524" layer="91"/>
+<wire x1="180.34" y1="137.16" x2="203.2" y2="137.16" width="0.1524" layer="91"/>
+<wire x1="203.2" y1="137.16" x2="203.2" y2="154.94" width="0.1524" layer="91"/>
+<pinref part="U3" gate="G$1" pin="CSB@2"/>
+<wire x1="203.2" y1="154.94" x2="208.28" y2="154.94" width="0.1524" layer="91"/>
+<wire x1="203.2" y1="154.94" x2="203.2" y2="160.02" width="0.1524" layer="91"/>
+<junction x="203.2" y="154.94"/>
+<pinref part="U3" gate="G$1" pin="CSB@1"/>
+<wire x1="203.2" y1="160.02" x2="208.28" y2="160.02" width="0.1524" layer="91"/>
+<pinref part="C9" gate="G$1" pin="2"/>
+<wire x1="180.34" y1="139.7" x2="180.34" y2="137.16" width="0.1524" layer="91"/>
+<junction x="180.34" y="137.16"/>
+</segment>
+</net>
+<net name="SENSE_SDA" class="0">
+<segment>
+<pinref part="U2" gate="A" pin="SDA"/>
+<wire x1="76.2" y1="170.18" x2="96.52" y2="170.18" width="0.1524" layer="91"/>
+<label x="93.98" y="170.18" size="1.778" layer="95"/>
+</segment>
+<segment>
+<pinref part="U3" gate="G$1" pin="SDI/SDA"/>
+<wire x1="243.84" y1="170.18" x2="266.7" y2="170.18" width="0.1524" layer="91"/>
+<label x="261.62" y="170.18" size="1.778" layer="95"/>
+</segment>
+</net>
+<net name="SENSE_SCL" class="0">
+<segment>
+<pinref part="U2" gate="A" pin="SCL"/>
+<wire x1="76.2" y1="165.1" x2="96.52" y2="165.1" width="0.1524" layer="91"/>
+<label x="93.98" y="165.1" size="1.778" layer="95"/>
+</segment>
+<segment>
+<pinref part="U3" gate="G$1" pin="SCLK"/>
+<wire x1="243.84" y1="165.1" x2="266.7" y2="165.1" width="0.1524" layer="91"/>
+<label x="261.62" y="165.1" size="1.778" layer="95"/>
+</segment>
+</net>
