File: eagle/projects/msp430_host_board/dacqs_host_board.sch (EAGLE design)
At the start: 215 parts, among them J1 MOL-SL-4-RA, J10 MOL-SL-3-V, J13 JST-PH-2TH-RA, J14 USB_MICROB_RECPT, J16 MOL-SL-2-RA, J17 CLM-112-02-L-D-IMU-MOUNT_IMU, J18 MOLSL-7-RA, J2 MOL-SL-4-RA, J3 MOL-SL-4-RA, J4 MOL-SL-4-RA, J5 MOL-SL-5-RA, J6 MOL-SL-3-V, J7 MOL-SL-5-V, J8 MOL-SL-3-RA, J9 MOL-SL-4-RA, U1 MSP430FR4994, U10 LSM9DS1, U2 MSP430FR4994, U3 PCT2075D,118, U4 MS560702BA03-50, U5 TPS61240DRVR, U6 LP5907_DBV_5, U7 MCP73831T, U8 INA219AIDCNR, U9 STD12NF06LT4, Y1 32.768kHz, Y3 32.768kHz

Commit message: Small changes to schematic
Parts:
- removed J11: (no value), daqcs_host:M02PTH
- added C35: 10uF, daqcs_host:CAP_10UF0_0603
- added C36: 100nF, daqcs_host:CAP_100NF0_0603
- added C37: 1uF, daqcs_host:CAP_1UF0_0603
- added R28: 10k, daqcs_host:RES_10R0_0603
Connections:
- net N$37 renamed TPS6_L
- removed net IMU_RST_2: J11.1, J17.8
- net +3V3: now also C35.1, C36.1, C37.1
- net CUTDOWN_EN: now also R28.2
- net GND: now also C35.2, C36.2, C37.2, R28.1
- net IMU_RST_1: now also J17.8; no longer J11.2
Other:
- moved on the sheet: C10, C6, C7, C8, C9
