File: eagle/projects/raspi_zero_power_sensor_hat/raspi_zero_power_sensor_hat.sch (EAGLE design)
At the start: 71 parts, among them J1 JST-PH-2TH-RA, J2 USB_MICROB_RECPT, J3 HEADER-1x2-2.54MM, J4 MOL-KK-2-V, J5 RECEPTACLE-2x7-2.54MM, J6 MOL-KK-4-RA, J7 MOL-KK-3P-V, J8 HEADER-1x4-2.54mm, Q1 PMOS-ENHANCE-8A, Q2 PMOS-ENHANCE-8A, U1 BUFFER-1-SCHMITT, U2 TPS61089RNRR, U3 INA219AIDCNR, U4 MCP73831T, U5 MS560702BA03-50, U6 PCT2075D,118, U7 SSCMNNN015PA2A3, U8 MAX11613EUA+

Commit message: final schematic without block diagram
Parts:
- removed R22: 10k, daqcs:RES_10R0_0603
- added NC1, NC2, NC3, NC4, NC5, NC6, NC7, NC8: NC, daqcs:NO_CONNECT
- added TP1, TP2, TP3, TP4, TP5, TP6, TP7: (no value), daqcs:TEST_POINT_TP10R_SMD_10R_SMD
- J8: value HEADER-1x4-2.54mm -> HEADER-1X5-2.54MM; device daqcs:HEADER-1X4-254MM_1X4_254MM_TH -> daqcs:HEADER-1X5-254MM_1X5_254MM_TH
Connections:
- new net N$10: J2.D-, NC6.NC
- new net N$11: J2.D+, NC7.NC
- new net N$12: J2.ID, NC8.NC
- new net N$4: NC1.NC, U5.SDO
- new net N$6: NC2.NC, U7.NC@1
- new net N$7: NC3.NC, U7.NC@2
- new net N$8: NC4.NC, U7.NC@3
- new net N$9: NC5.NC, U7.NC@4
- new net RASPI_GPIO17: J5.GPIO17/GPIO_GEN0, TP3.TP
- new net RASPI_GPIO18: J5.GPIO18/GPIO_GEN1/PWM0, TP2.TP
- new net RASPI_GPIO27: J5.GPIO27/GPIO_GEN2, TP4.TP
- net GND: now also J8.5
- net MCU_POWER_OFF: now also TP6.TP
- net PP3V3_RASPI: no longer R22.2
- net PP5V0_BOOST: now also TP5.TP
- net TEMP_I2C_ALERT: now also TP1.TP; no longer J5.GPIO17/GPIO_GEN0, R22.1
- net UART_RASPI_TXD_MCU_RXD: now also TP7.TP

Commit message: finalized schematic
Connections:
- net MCU_POWER_OFF: no longer TP6.TP
- net UART_RASPI_RXD_MCU_TXD: now also TP6.TP
Other:
- moved on the sheet: TP6
Changed lines of the file:
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@@
 <part name="NC8" library="daqcs" deviceset="NO_CONNECT" device="" value="NC"/>
 <part name="FRAME2" library="daqcs" deviceset="FRAME_B_L" device=""/>
+<part name="U$1" library="daqcs" deviceset="BLOCK_DIAGRAM" device=""/>
 </parts>
 <sheets>
@@
 <instance part="FRAME2" gate="G$1" x="0" y="0"/>
 <instance part="FRAME2" gate="G$2" x="325.8312" y="0.4572"/>
+<instance part="U$1" gate="G$1" x="28.448" y="30.988"/>
 </instances>
 <busses>
@@
 <text x="180.34" y="53.34" size="1.778" layer="91">Charger Status LEDs</text>
 <text x="421.64" y="7.62" size="3.81" layer="91">A</text>
-<text x="330.2" y="27.94" size="3.81" layer="91">PI_MCU_CONNECT_AND_SENSORS</text>
+<text x="330.2" y="27.94" size="3.81" layer="91">POWER_ENTRY_BOOST_CHARGER</text>
 <text x="144.78" y="226.06" size="1.778" layer="91">Vin UVLO: 2.5V (MAX)</text>
 <text x="317.5" y="86.36" size="1.778" layer="91">Vt+: 2.79V (MAX)</text>
@@
 <attribute name="TP_SIGNAL_NAME" x="16.51" y="196.85" size="1.778" layer="97" rot="R90"/>
 </instance>
-<instance part="TP6" gate="G$1" x="78.74" y="149.86"/>
+<instance part="TP6" gate="G$1" x="93.98" y="149.86"/>
 <instance part="TP7" gate="G$1" x="86.36" y="149.86"/>
 <instance part="NC1" gate="G$1" x="284.48" y="190.5" rot="R180"/>
@@
 <label x="48.26" y="134.62" size="1.778" layer="95"/>
 <pinref part="TP7" gate="G$1" pin="TP"/>
-<wire x1="86.36" y1="134.62" x2="93.98" y2="134.62" width="0.1524" layer="91"/>
+<wire x1="86.36" y1="134.62" x2="99.06" y2="134.62" width="0.1524" layer="91"/>
 <wire x1="86.36" y1="144.78" x2="86.36" y2="134.62" width="0.1524" layer="91"/>
 <junction x="86.36" y="134.62"/>
@@
 <wire x1="38.1" y1="124.46" x2="93.98" y2="124.46" width="0.1524" layer="91"/>
 <label x="48.26" y="124.46" size="1.778" layer="95"/>
+<pinref part="TP6" gate="G$1" pin="TP"/>
+<wire x1="93.98" y1="124.46" x2="99.06" y2="124.46" width="0.1524" layer="91"/>
+<wire x1="93.98" y1="144.78" x2="93.98" y2="124.46" width="0.1524" layer="91"/>
+<junction x="93.98" y="124.46"/>
 </segment>
 </net>
@@
 <segment>
 <pinref part="J6" gate="G$1" pin="1"/>
-<wire x1="38.1" y1="139.7" x2="78.74" y2="139.7" width="0.1524" layer="91"/>
+<wire x1="38.1" y1="139.7" x2="99.06" y2="139.7" width="0.1524" layer="91"/>
 <label x="48.26" y="139.7" size="1.778" layer="95"/>
-<pinref part="TP6" gate="G$1" pin="TP"/>
-<wire x1="78.74" y1="139.7" x2="93.98" y2="139.7" width="0.1524" layer="91"/>
-<wire x1="78.74" y1="144.78" x2="78.74" y2="139.7" width="0.1524" layer="91"/>
-<junction x="78.74" y="139.7"/>
-</segment>
-</net>
+</segment>
+</net>

Commit message: modified cap and res to have more attributes
Parts:
- removed H4: MOUNT-HOLE_2.75, daqcs:MOUNT-HOLE_2.75
Connections:
- net GND: now also C12.2; no longer C12.1
- net PP5V0_BOOST: now also C12.1; no longer C12.2
Other:
- moved on the sheet: C1, C10, C11, C12, C14, C16, C18, C3, C4, C5, C7, C8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

Commit message: modified pi hat schematic. Added second temp sensor. Removed Honeywell pressure sensor for two TE sensors
Parts:
- removed H1, H2, H3: MOUNT-HOLE_2.75, daqcs:MOUNT-HOLE_2.75
- removed J6: MOL-KK-4-RA, daqcs:MOLKK_4PIN_4RA_RA
- removed J7: MOL-KK-3P-V, daqcs:MOLKK_3PIN_3V_V
- removed NC4, NC5: NC, daqcs:NO_CONNECT
- removed R23, R24: 2k, daqcs:RES_2R0_0603
- removed R25: 4.7k, daqcs:RES_4R7_0603
- removed TP3, TP4, TP6, TP7: (no value), daqcs:TEST_POINT_TP10R_SMD_10R_SMD
- added C20: 100nF, daqcs:CAP_100NF0_0603
- added DS7, DS8: GREEN, daqcs:LED_G3V2WURTH_0603
- added H4, H5, H6: MOUNT-HOLE_2.75, daqcs:MOUNT-HOLE_2.75
- added J10: MOL-SL-4-V, daqcs:MOLSL_4PIN_SL4V_V
- added J11: MOL-SL-3-V, daqcs:MOLSL_3PIN_SL3V_V
- added J9: RECEPTACLE-2x7-2.54MM, daqcs:RECEPTICAL-2X7-254MM-PIZERO_2X7_254MM_TH
- added R19: 0, daqcs:RES_0R0_0603
- added R20, R22, R30, R31, R5: 2k, daqcs:RES_2R0_0603
- added R26: 4.7k, daqcs:RES_4R7_0603
- added TP10, TP11, TP12, TP8, TP9: (no value), daqcs:TEST_POINT_TP10R_SMD_10R_SMD
- added U9: PCT2075D,118, daqcs:PCT2075D,118SOIC8
- J1: value JST-PH-2TH-RA -> MOL-SL-2-RA; device daqcs:JST-PH-2TH-RA_2TH-RA -> daqcs:MOLSL_2PIN_SL2RA_RA
- J4: value MOL-KK-2-V -> MOL-SL-2-V; device daqcs:MOLKK_2PIN2V_2V -> daqcs:MOLSL_2PIN_SL2V_V
- J5: value RECEPTACLE-2x7-2.54MM -> HEADER-1x4-2.54mm; device daqcs:RECEPTICAL-2X7-254MM-PIZERO_2X7_254MM_TH -> daqcs:HEADER-1X4-254MM_1X4_254MM_TH
- R12, R13: value 1k -> 2k; device daqcs:RES_1R0_0603 -> daqcs:RES_2R0_0603
- R14: value 1k -> 0; device daqcs:RES_1R0_0603 -> daqcs:RES_0R0_0603
- U7: value SSCMNNN015PA2A3 -> MS580305BA01; device daqcs:SSCMNNN015PA2A3_8SMD -> daqcs:MS5803-05BA_8SMD
Connections:
- net MS_CSB renamed PRES0_CSB
- net TEMP_I2C_A0 renamed TEMP0_I2C_A0
- net TEMP_I2C_ALERT renamed TEMP0_I2C_ALERT
- removed net N$6: NC2.NC, U7.NC@1
- removed net N$9: NC5.NC, U7.NC@4
- new net DBG_LED0: DS7.C, R30.2
- new net DBG_LED1: DS8.C, R31.2
- new net N$2: U9.A1
- new net PRES1_CSB: R19.1, U7.CSB
- new net TEMP1_I2C_A0: R14.2, U9.A0
- new net TEMP1_I2C_ALERT: TP2.TP, U9.OS
- net BOOST_PG: now also R12.2; no longer R13.2
- net BOOST_SW_PG: now also R13.2; no longer R14.2
- net CHG_DONE: now also R5.2; no longer R12.2
- net GND: now also C15.1, C18.1, C20.2, J10.3, J11.2, J5.4, J9.GND@1, J9.GND@2, J9.GND@3, R30.1, R31.1, R5.1, U9.A2, U9.GND; no longer C15.2, C18.2, J1.2, J5.GND@1, J5.GND@2, J5.GND@3, J6.3, J7.2
- net I2C1_RASPI_SCL: now also J5.3, J9.GPIO3/SCL1, R20.1, U7.SCLK, U9.SCL; no longer J5.GPIO3/SCL1, R23.1, U7.SCL
- net I2C1_RASPI_SDA: now also J5.2, J9.GPIO2/SDA1, R22.1, U7.SDI/SDA, U9.SDA; no longer J5.GPIO2/SDA1, R24.1, U7.SDA
- net MCU_POWER_OFF: now also J10.1; no longer J6.1
- net N$7: now also NC2.NC, U7.SDO; no longer NC3.NC, U7.NC@2
- net N$8: now also NC3.NC, U7.NC; no longer NC4.NC, U7.NC@3
- net PP3V3_RASPI: now also C15.2, C18.2, C20.1, J11.1, J5.1, J9.3V3, R19.2, R20.2, R22.2, R26.2, U7.PS, U7.VDD, U9.VCC; no longer C15.1, C18.1, J5.3V3, J7.1, R23.2, R24.2, R25.2, U7.VCC
- net PP5V0_BOOST_SW: now also J9.5V0@1, J9.5V0@2; no longer J5.5V0@1, J5.5V0@2
- net RASPI_GPIO17: now also DS7.A, J9.GPIO17/GPIO_GEN0, TP9.TP; no longer J5.GPIO17/GPIO_GEN0, TP3.TP
- net RASPI_GPIO18: now also J9.GPIO18/GPIO_GEN1/PWM0, TP8.TP; no longer J5.GPIO18/GPIO_GEN1/PWM0, TP2.TP
- net RASPI_GPIO27: now also DS8.A, J9.GPIO27/GPIO_GEN2, TP10.TP; no longer J5.GPIO27/GPIO_GEN2, TP4.TP
- net TEMP_1WIRE_BI: now also J11.3, J9.GPIO4/GPIO_GCLK/1-WIRE, R26.1; no longer J5.GPIO4/GPIO_GCLK/1-WIRE, J7.3, R25.1
- net UART_RASPI_RXD_MCU_TXD: now also J10.4, J9.GPIO15/RXD0, TP11.TP; no longer J5.GPIO15/RXD0, J6.4, TP6.TP
- net UART_RASPI_TXD_MCU_RXD: now also J10.2, J9.GPIO14/TXD0, TP12.TP; no longer J5.GPIO14/TXD0, J6.2, TP7.TP
Other:
- note added: "3.3V Power"
- note added: "ADD 3.3V LDO HERE"
- note added: "Current/Voltage Sense Amp."
- note added: "DEBUG LEDs"
- note added: "HOST/RASPI CONNECTORS and MOUNTING"
- note added: "I2C Addr: 0x94/0x95 (W/R)"
- note added: "I2C Addr: 0xEC/0xED (W/R)"
- note added: "I2C DEBUG HEADER/PWR"
- note added: "MOUNTING HOLES"
- note added: "Only using 3 mounting holes since"
- note added: "PI_MCU_CONNECT_AND_MOUNTING"
- note added: "Pressure Sensor 0"
- note added: "Pressure Sensor 1"
- note added: "SENSORS"
- note added: "Temperature Sensor 0"
- note added: "Temperature Sensor 1"
- note added: "This allows for easier routing of the"
- note added: "boost output to the Pi's 5V0 pin."
- note added: "the 2x7 pin connector stabilizes"
- note added: "the upper left board quadrant."
- note removed: "(Honeywell)"
- note removed: "(TE)"
- note removed: "5.3V Power"
- note removed: "Current/Voltage"
- note removed: "HOST/RASPI CONNECTORS and SENSORS"
- note removed: "I2C Addr: 0x28/0x29 (W/R)"
- note removed: "PI_MCU_CONNECT_AND_SENSORS"
- note removed: "Pressure Sensor"
- note removed: "Sense Amplifier"
- note removed: "Temperature Sensor"

Commit message: added 3.3V LDO for non- RasPi operation
Parts:
- removed DS1: GREEN, daqcs:LED_G3V2WURTH_0603
- removed DS2: YELLOW, daqcs:LED_Y2V0WURTH_0603
- removed J2: USB_MICROB_RECPT, daqcs:USB_B_MICRO_RIGHT
- removed J4: MOL-SL-2-V, daqcs:MOLSL_2PIN_SL2V_V
- removed NC8: NC, daqcs:NO_CONNECT
- removed R10, R11: 2k, daqcs:RES_2R0_0603
- removed R15: 0, daqcs:RES_0R0_0603
- added C21: 10uF, daqcs:CAP_10UF0_0603
- added DS5: GREEN, daqcs:LED_G3V2WURTH_0603
- added DS6: YELLOW, daqcs:LED_Y2V0WURTH_0603
- added J6: USB_MICROB_RECPT, daqcs:USB_B_MICRO_RIGHT
- added J7: MOL-SL-2-V, daqcs:MOLSL_2PIN_SL2V_V
- added NC4, NC5, NC9: NC, daqcs:NO_CONNECT
- added R23, R24, R32: 2k, daqcs:RES_2R0_0603
- added R25: 0, daqcs:RES_0R0_0603
- added U10: MCP73831T, daqcs:MCP73831T-2ATI/OT
- C13: value 10uF -> 100nF; device daqcs:CAP_10UF0_0603 -> daqcs:CAP_100NF0_0603
- R5: value 2k -> 0; device daqcs:RES_2R0_0603 -> daqcs:RES_0R0_0603
- U4: value MCP73831T -> TLV71333P; device daqcs:MCP73831T-2ATI/OT -> daqcs:TLV71333PDBVR_SOT23
Connections:
- removed net N$11: J2.D+, NC7.NC
- removed net N$12: J2.ID, NC8.NC
- new net N$13: J6.D+, NC5.NC
- new net N$14: J6.ID, NC9.NC
- new net N$6: NC6.NC, U4.NC
- new net N$9: J6.D-, NC4.NC
- new net PP3V3_LDO: C13.1, R5.1, U4.OUT
- net CHG_DONE: now also DS5.C, R32.2; no longer DS1.C, R5.2
- net CHG_ON: now also DS6.A, R24.1; no longer DS2.A, R11.1
- net CHG_PROG: now also R23.2, U10.PROG; no longer R10.2, U4.PROG
- net CHG_STAT: now also DS5.A, DS6.C, U10.STAT; no longer DS1.A, DS2.C, U4.STAT
- net GND: now also C21.2, J6.GND, J7.2, R23.1, R25.1, R32.1, U10.VSS, U4.GND; no longer J2.GND, J4.2, R10.1, R15.1, R5.1, U4.VSS
- net N$10: now also NC7.NC, U1.NC; no longer J2.D-, NC6.NC
- net PP3V3_RASPI: now also R5.2
- net PP5V0_BOOST_SW: now also U4.EN, U4.IN
- net PP5V0_USB: now also C21.1, J6.5V, J7.1, R24.2, U10.VDD; no longer C13.1, J2.5V, J4.1, R11.2, U4.VDD
- net USB_SHD: now also J6.SLD, R25.2; no longer J2.SLD, R15.2
- net VBAT: now also U10.VBAT; no longer U4.VBAT
Other:
- note added: "1.00k --> 1000mA"
- note added: "1.33k --> 750mA"
- note added: "2.00k --> 500mA"
- note added: "3.3V LDO (No RasPi Operation)"
- note added: "5V Charger Input"
- note added: "ADD HUMIDITY SENSOR HERE"
- note added: "ADD WATCHDOG"
- note added: "Charger"
- note added: "DO NOT connect both"
- note added: "I2C DEBUG HEADER"
- note added: "LEDs"
- note added: "LIPO_CHARGER"
- note added: "LiPo Charger"
- note added: "POWER ENTRY, 5V BOOST, AND 3.3V LDO"
- note added: "POWER_ENTRY_BOOST_LDO"
- note added: "Placeholder for 3.3V rail supply if the"
- note added: "RASPI SBC MOUNTING HOLES"
- note added: "RasPi supplies the 3.3V rail during operation"
- note added: "Status"
- note added: "USB or Benchtop"
- note added: "board is used without a RasPi, since the"
- note added: "current limit:"
- note removed: "ADD 3.3V LDO HERE"
- note removed: "Charger Status LEDs"
- note removed: "I2C DEBUG HEADER/PWR"
- note removed: "MOUNTING HOLES"
- note removed: "POWER ENTRY, 5V BOOST, AND CHARGER"
- note removed: "POWER_ENTRY_BOOST_CHARGER"
- note removed: "current limit = 500mA"
