File: eagle/projects/raspi_zero_power_sensor_hat/raspi_zero_power_sensor_hat.sch (EAGLE design)
At the start: 106 parts, among them J1 MOL-SL-2-RA, J10 MOL-SL-4-V, J11 MOL-SL-3-V, J2 RECEPTACLE-2x3-2.54MM, J3 HEADER-1x2-2.54MM, J4 MOL-SL-5-V, J5 HEADER-1x4-2.54mm, J6 SI7021, J7 MOL-SL-2-V, J9 RECEPTACLE-2x7-2.54MM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

Commit message: using a 2x6 pin header to connecting to the RasPi instead of 2x7. THis saves room and only removes a debug pin and GND pin. THis is fine since the RUN pin header adds 2 more GPIO plus 1 GND. added notes for male pin headers that mate to the 2x6 and RUN pin headers. fixed silk on all rectangular headers
Parts:
- removed J9: RECEPTACLE-2x7-2.54MM, daqcs:RECEPTICAL-2X7-254MM-PIZERO_2X7_254MM_TH
- removed TP10: (no value), daqcs:TEST_POINT_TP10R_SMD_10R_SMD
- added J8: RECEPTACLE-2x6-2.54MM, daqcs:RECEPTICAL-2X6-254MM-PIZERO_2X6_254MM_TH
Connections:
- removed net RASPI_GPIO21: J2.GPIO21/SCLK, TP4.TP
- removed net RASPI_GPIO27: DS8.A, J9.GPIO27/GPIO_GEN2, TP10.TP
- new net RASPI_GPIO18: DS8.A, J8.GPIO18/GPIO_GEN1/PWM0, TP4.TP
- net ADC_AIN0: now also J4.4; no longer J4.1
- net ADC_AIN1: now also J4.3; no longer J4.2
- net ADC_AIN2: now also J4.2; no longer J4.3
- net ADC_AIN3_REF: now also J4.1; no longer J4.4
- net GND: now also J8.GND@1, J8.GND@2; no longer J9.GND@1, J9.GND@2, J9.GND@3
- net I2C1_RASPI_SCL: now also J8.GPIO3/SCL1; no longer J9.GPIO3/SCL1
- net I2C1_RASPI_SDA: now also J8.GPIO2/SDA1; no longer J9.GPIO2/SDA1
- net PP3V3_RASPI: now also J8.3V3; no longer J9.3V3
- net PP5V0_BOOST_SW: now also J8.5V0@1, J8.5V0@2; no longer J9.5V0@1, J9.5V0@2
- net RASPI_GPIO17: now also J8.GPIO17/GPIO_GEN0; no longer J9.GPIO17/GPIO_GEN0
- net TEMP_1WIRE_BI: now also J8.GPIO4/GPIO_GCLK/1-WIRE; no longer J9.GPIO4/GPIO_GCLK/1-WIRE
- net UART_RASPI_RXD_MCU_TXD: now also J8.GPIO15/RXD0; no longer J9.GPIO15/RXD0
- net UART_RASPI_TXD_MCU_RXD: now also J8.GPIO14/TXD0; no longer J9.GPIO14/TXD0
- net WDT_PET: now also J2.GPIO21/SCLK; no longer J9.GPIO18/GPIO_GEN1/PWM0
Other:
- note added: "DEBUG LED"
- note added: "Digi-Key PN: 952-2120-ND"
- note added: "Digi-Key PN: 952-2125-ND"
- note added: "Harwin PN: M20-9980345"
- note added: "Harwin PN: M20-9980645"
- note added: "Mates with 2x3 pin header on RasPi"
- note added: "Mates with 2x6 pin header on RasPi"
- note added: "across 40-pin header pins 1-14"
- note added: "across the RUN header and 40-pin header"
- note removed: "DEBUG LEDs"
- moved on the sheet: DS7, DS8, R30, R31, TP4

Commit message: added inverting OD buffer so that the MSP can drive the RUN pin on the Pi. This allows the MSP to either cycle all RasPi power or just hard reset the BCM (note this is done through a stuff option, cant use both methods)
Parts:
- added C22: 100nF, daqcs:CAP_100NF0_0603
- added NC9: NC, daqcs:NO_CONNECT
- added U1: INV-1-SCHMITT, daqcs:INVERTER-1-SCHMITT_INV1_TSSOP5
Connections:
- new net N$10: NC9.NC, U1.NC
- net GND: now also C22.2, U1.GND
- net MCU_POWER_OFF: now also U1.A
- net PP3V3_RASPI: now also C22.1, U1.VCC
- net WDT_BITE_N: now also U1.Y
Other:
- note added: "(includes sensors, PMU, and BCM2835)"
- note added: "RESET_AND_LIPO_CHARGER"
- note added: "Reset Circuitry and LiPo Battery Charger"
- note removed: "LiPo Battery Charger and Reset Circuitry"
- moved on the sheet: C21, C23, C24, DS5, DS6, J7, NC5, NC8, R17, R23, R24, R25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

Commit message: corrected mounting holes for RasPi and Cam. added the correct holes to the schematic. TO DO: make a template part that has the correct HAT outline and mounting holes for the external 3 standoffs
Parts:
- added H1, H2, H3: 2.75mm_drill_3.00mm_radius, daqcs:MOUNT-HOLE_2.75_3.0
- added H7: 2.2mm_drill_2.0mm_radius, daqcs:MOUNT-HOLE_2.2_2.0
- H4, H5, H6: value MOUNT-HOLE_2.75 -> 2.2mm_drill_2.0mm_radius; device daqcs:MOUNT-HOLE_2.75 -> daqcs:MOUNT-HOLE_2.2_2.0
Other:
- note added: "MAKE A TEMPLATE PART"
- note added: "WHICH HAS HAT OUTLINE AND MOUNTING HOLES"
- moved on the sheet: H4, H5, H6
Changed lines of the file:
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@@
 <part name="C20" library="daqcs" deviceset="CAP" device="_0603" technology="_100NF0" value="100nF"/>
 <part name="GND46" library="daqcs" deviceset="GND" device=""/>
-<part name="H4" library="daqcs" deviceset="MOUNT-HOLE" device="_2.75"/>
-<part name="H5" library="daqcs" deviceset="MOUNT-HOLE" device="_2.75"/>
-<part name="H6" library="daqcs" deviceset="MOUNT-HOLE" device="_2.75"/>
 <part name="TP9" library="daqcs" deviceset="TEST_POINT" device="_10R_SMD" technology="_TP10R_SMD"/>
 <part name="TP11" library="daqcs" deviceset="TEST_POINT" device="_10R_SMD" technology="_TP10R_SMD"/>
@@
 <part name="NC9" library="daqcs" deviceset="NO_CONNECT" device="" value="NC"/>
 <part name="PP3V3_RASPI14" library="daqcs" deviceset="PP3V3_RASPI" device=""/>
+<part name="H1" library="daqcs" deviceset="MOUNT-HOLE" device="_2.75_3.0" value="2.75mm_drill_3.00mm_radius"/>
+<part name="H2" library="daqcs" deviceset="MOUNT-HOLE" device="_2.75_3.0" value="2.75mm_drill_3.00mm_radius"/>
+<part name="H3" library="daqcs" deviceset="MOUNT-HOLE" device="_2.75_3.0" value="2.75mm_drill_3.00mm_radius"/>
+<part name="H4" library="daqcs" deviceset="MOUNT-HOLE" device="_2.2_2.0" value="2.2mm_drill_2.0mm_radius"/>
+<part name="H5" library="daqcs" deviceset="MOUNT-HOLE" device="_2.2_2.0" value="2.2mm_drill_2.0mm_radius"/>
+<part name="H6" library="daqcs" deviceset="MOUNT-HOLE" device="_2.2_2.0" value="2.2mm_drill_2.0mm_radius"/>
+<part name="H7" library="daqcs" deviceset="MOUNT-HOLE" device="_2.2_2.0" value="2.2mm_drill_2.0mm_radius"/>
 </parts>
 <sheets>
@@
 <instance part="GND59" gate="1" x="91.44" y="142.24"/>
 <instance part="R33" gate="G$1" x="106.68" y="172.72" rot="R180"/>
-<instance part="U13" gate="G$1" x="340.36" y="198.12"/>
+<instance part="U13" gate="G$1" x="340.36" y="198.12">
+<attribute name="OUTPUT_TYPE" x="335.28" y="180.34" size="1.778" layer="96"/>
+</instance>
 <instance part="R35" gate="G$1" x="297.18" y="182.88" rot="R90"/>
 <instance part="GND60" gate="1" x="297.18" y="170.18"/>
 <instance part="GND61" gate="1" x="325.12" y="180.34"/>
 <instance part="NC8" gate="G$1" x="358.14" y="187.96" rot="R180"/>
-<instance part="U1" gate="G$1" x="360.68" y="121.92"/>
+<instance part="U1" gate="G$1" x="360.68" y="121.92">
+<attribute name="OUTPUT_TYPE" x="355.6" y="104.14" size="1.778" layer="96"/>
+</instance>
 <instance part="C22" gate="G$1" x="332.74" y="137.16"/>
 <instance part="GND39" gate="1" x="332.74" y="127"/>
@@
 <text x="71.12" y="210.82" size="1.778" layer="91" rot="R90">NOSTUFF</text>
 <text x="175.26" y="149.86" size="2.54" layer="91">DEBUG LED</text>
+<text x="66.04" y="17.78" size="3.81" layer="91">MAKE A TEMPLATE PART</text>
+<text x="66.04" y="12.7" size="3.81" layer="91">WHICH HAS HAT OUTLINE AND MOUNTING HOLES</text>
 </plain>
 <instances>
@@
 </instance>
 <instance part="GND46" gate="1" x="317.5" y="154.94"/>
-<instance part="H4" gate="G$1" x="43.18" y="58.42"/>
-<instance part="H5" gate="G$1" x="43.18" y="50.8"/>
-<instance part="H6" gate="G$1" x="43.18" y="43.18"/>
 <instance part="TP9" gate="G$1" x="38.1" y="182.88" smashed="yes" rot="R90">
 <attribute name="NAME" x="31.75" y="182.88" size="1.778" layer="95" rot="R180" align="center"/>
@@
 <instance part="GND20" gate="1" x="205.74" y="142.24"/>
 <instance part="J8" gate="G$1" x="137.16" y="195.58"/>
+<instance part="H1" gate="G$1" x="40.64" y="55.88"/>
+<instance part="H2" gate="G$1" x="40.64" y="48.26"/>
+<instance part="H3" gate="G$1" x="40.64" y="40.64"/>
+<instance part="H4" gate="G$1" x="160.02" y="58.42"/>
+<instance part="H5" gate="G$1" x="160.02" y="50.8"/>
+<instance part="H6" gate="G$1" x="160.02" y="43.18"/>
+<instance part="H7" gate="G$1" x="160.02" y="35.56"/>
 </instances>
 <busses>

Commit message: renamed file name for Honey sensor... for steve
Other:
- note added: "RASPBERRY PI RESET/GPIO HEADER"
- moved on the sheet: C12, C16, C18, C2, J6, NC4, NC7, R14, R21, R4, TP1, TP2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
