File: eagle/projects/raspi_zero_power_sensor_hat/raspi_zero_power_sensor_hat.brd (EAGLE design)
At the start: 304.5 x 229.3 mm, 156 parts, among them J301 MOL-SL-2-V, J302 USB_MICROB_RECPT, J401 MOL-SL-2-RA, J501 MOL-SL-5-V, J601 RECEPTACLE-2x6-2.54MM, J602 HEADER-1x4-2.54mm, J603 MOL-SL-4-V, J604 RECEPTACLE-2x3-2.54MM, J605 MOL-SL-3-V, Q301 NMOS-DUAL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

Commit message: Fixed all schematic ERCs except for IMU and Humidity sensor. Changed all power line jumpers to 0805
Parts:
- Q301, Q401: value NMOS-DUAL -> SSM6N7002KFU
- R402, R607: device daqcs:R0603 -> daqcs:R0805
- R403: value 49.9k -> 49.9
- moved R403 384.4 mm to (-117.6, -264.9)
- moved R402 375.4 mm to (-121.7, -263.8)
- moved R607 344.3 mm to (-124.9, -263.8)
Connections:
- net 3V3_PG renamed 3V3_HAT_PG
- net BOOST_SW_PG renamed 5V0_BST_PG
- net MCU_TO_BOOST_RESET renamed MCU_TO_BST_RESET
- net N$4 renamed USB_SHD
- removed net N$1: C404.1, Q401.2, R403.1, R406.2
- new net CHG_DISABLE_GATE: C404.1, Q401.2, R403.2, R406.2
- net GND: now also J605.3; no longer J605.2
- net PP5V0_CHG_IN: now also R403.1; no longer R403.2
- net TEMP_1WIRE_BI: now also J605.2; no longer J605.3
- net TEMP_1WIRE_BI_R: now also R606.2

Commit message: added 0-ohms to the unused mosfet, as per Mark's request
Parts:
- added R311: 10k, daqcs:R0603
- added R312: 49.9, daqcs:R0603
- R307, R308: value 10k -> 0.0
- R310: value 49.9 -> 10k
- moved R306 402.6 mm to (-124.0, -270.1)
- moved R307 363.0 mm to (-114.4, -228.6)
- moved R310 125.7 mm to (32.7, 82.4)
- moved R308 109.2 mm to (133.2, 39.6)
- moved R305 40.1 mm to (-124.0, -267.5)
- moved R309 2.30 mm to (133.2, 36.9)
Connections:
- new net N$1: Q301.3, R305.2
- new net N$2: Q301.5, R305.1, R306.1
- net GND: now also R306.2, R309.1, R310.1; no longer Q301.3, Q301.5, R307.1, R308.1
- net MCU_TO_RASPI_RESET: now also R310.2; no longer R308.2
- net PP3V3_HAT: now also R308.2, R311.2; no longer R306.2, R309.2
- net RASPI_RESET_N: now also R312.2; no longer R310.2
- net RESET_BITE_N: now also R311.1, R312.1; no longer R309.1, R310.1
- net WDT_PET: now also R309.2; no longer R305.2
- net WDT_PET_R: now also R307.1; no longer R305.1
- net WDT_SET2: now also R308.1; no longer R306.1

Commit message: swapped battery charger for AC variant. Checked charger symbol and footprint :)
Parts:
- U301: value MCP73831T -> MCP73831T-2AC
- moved U301 401.0 mm to (-123.3, -273.8)
Changed lines of the file:
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@@
 <attribute name="DATASHEET" value="HW/docs/projects/raspi_zero_power_sensor_hat/datasheets/sensors/ENG_DS_MS5803-05BA_B.pdf" x="128.47" y="76.76" size="1.778" layer="27" display="off"/>
-</element>
-<element name="U301" library="daqcs" package="SOT23P110X060-5N" value="MCP73831T" x="120.75" y="44.45">
-<attribute name="VENDOR_PN" value="MCP73831T-2ATI/OTCT-ND" x="101.86" y="62.45" size="1.778" layer="27" display="off"/>
-<attribute name="VENDOR" value="Digi-key" x="101.86" y="62.45" size="1.778" layer="27" display="off"/>
-<attribute name="MANUFACTURER_PN" value="MCP73831T-2ATI/OT" x="101.86" y="62.45" size="1.778" layer="27" display="off"/>
-<attribute name="MANUFACTURER" value="Microchip" x="101.86" y="62.45" size="1.778" layer="27" display="off"/>
-<attribute name="DATASHEET" value="HW/docs/projects/raspi_zero_power_sensor_hat/datasheets/charger/20001984g.pdf" x="120.75" y="44.45" size="1.778" layer="27" display="off"/>
 </element>
 <element name="R302" library="daqcs" package="R0603" value="2k" x="117.06" y="35.73">
@@
 <attribute name="TOLERANCE" value="Jumper" x="-124" y="-270.09" size="1.778" layer="27" display="off"/>
 <attribute name="VENDOR" value="Digi-key" x="-124" y="-270.09" size="1.778" layer="27" display="off"/>
+</element>
+<element name="U301" library="daqcs" package="SOT23P110X060-5N" value="MCP73831T-2AC" x="-123.28" y="-273.76">
+<attribute name="VENDOR" value="Digi-key" x="-123.28" y="-273.76" size="1.778" layer="27" display="off"/>
+<attribute name="DATASHEET" value="HW/docs/projects/raspi_zero_power_sensor_hat/datasheets/charger/20001984g.pdf" x="-123.28" y="-273.76" size="1.778" layer="27" display="off"/>
+<attribute name="VENDOR_PN" value="MCP73831T-2ACI/OTCT-ND" x="-123.28" y="-273.76" size="1.778" layer="27" display="off"/>
+<attribute name="MANUFACTURER_PN" value="MCP73831T-2ACI/OT" x="-123.28" y="-273.76" size="1.778" layer="27" display="off"/>
+<attribute name="MANUFACTURER" value="Microchip" x="-123.28" y="-273.76" size="1.778" layer="27" display="off"/>
 </element>
 </elements>
@@
 <contactref element="U507" pad="2"/>
 <contactref element="R304" pad="1"/>
-<contactref element="U301" pad="2"/>
 <contactref element="C301" pad="2"/>
 <contactref element="J301" pad="2"/>
@@
 <contactref element="J605" pad="3"/>
 <contactref element="R306" pad="2"/>
+<contactref element="U301" pad="2"/>
 <wire x1="146.1" y1="88.685" x2="148.7" y2="89.985" width="0" layer="19" extent="1-1"/>
 <wire x1="143.99" y1="86.1" x2="146.1" y2="88.685" width="0" layer="19" extent="1-1"/>
@@
 <wire x1="113.61" y1="34.99" x2="116.21" y2="35.73" width="0" layer="19" extent="1-1"/>
 <wire x1="113.13" y1="43.63" x2="116.21" y2="35.73" width="0" layer="19" extent="1-1"/>
-<wire x1="119.35" y1="44.45" x2="113.13" y2="43.63" width="0" layer="19" extent="1-1"/>
 <wire x1="152" y1="40.74" x2="134.14" y2="42.2" width="0" layer="19" extent="1-1"/>
 <wire x1="152" y1="47.24" x2="152" y2="40.74" width="0" layer="19" extent="1-1"/>
@@
 <wire x1="-118.45" y1="-262.47" x2="-118.45" y2="-260.16" width="0" layer="19" extent="1-1"/>
 <wire x1="-123.15" y1="-270.09" x2="-118.45" y2="-262.47" width="0" layer="19" extent="1-1"/>
+<wire x1="-124.68" y1="-273.76" x2="-123.15" y2="-270.09" width="0" layer="19" extent="1-1"/>
 </signal>
 <signal name="VBAT">
 <contactref element="C401" pad="1"/>
 <contactref element="J401" pad="1"/>
-<contactref element="U301" pad="3"/>
 <contactref element="TP401" pad="TP"/>
 <contactref element="R401" pad="2A"/>
-<wire x1="19.46" y1="82.41" x2="119.35" y2="43.5" width="0" layer="19" extent="1-1"/>
+<contactref element="U301" pad="3"/>
+<wire x1="13.75" y1="12.18" x2="-124.68" y2="-274.71" width="0" layer="19" extent="1-1"/>
+<wire x1="19.46" y1="82.41" x2="13.75" y2="12.18" width="0" layer="19" extent="1-1"/>
 <wire x1="19.99" y1="87.68" x2="19.46" y2="82.41" width="0" layer="19" extent="1-1"/>
 <wire x1="19.595" y1="89.67" x2="19.99" y2="87.68" width="0" layer="19" extent="1-1"/>
-<wire x1="13.75" y1="12.18" x2="19.46" y2="82.41" width="0" layer="19" extent="1-1"/>
 </signal>
 <signal name="VBAT_SNS_P">
@@
 </signal>
 <signal name="CHG_STAT">
-<contactref element="U301" pad="1"/>
 <contactref element="DS301" pad="1"/>
 <contactref element="DS302" pad="2"/>
 <contactref element="TP302" pad="TP"/>
-<wire x1="119.35" y1="45.4" x2="123.44" y2="40.4" width="0" layer="19" extent="1-1"/>
-<wire x1="123.2" y1="37.45" x2="119.35" y2="45.4" width="0" layer="19" extent="1-1"/>
-<wire x1="119.28" y1="40.64" x2="123.2" y2="37.45" width="0" layer="19" extent="1-1"/>
+<contactref element="U301" pad="1"/>
+<wire x1="123.2" y1="37.45" x2="123.44" y2="40.4" width="0" layer="19" extent="1-1"/>
+<wire x1="119.28" y1="40.64" x2="123.44" y2="40.4" width="0" layer="19" extent="1-1"/>
+<wire x1="-124.68" y1="-272.81" x2="123.2" y2="37.45" width="0" layer="19" extent="1-1"/>
 </signal>
 <signal name="CHG_DONE">
@@
 </signal>
 <signal name="CHG_PROG">
+<contactref element="R302" pad="2"/>
 <contactref element="U301" pad="5"/>
-<contactref element="R302" pad="2"/>
-<wire x1="122.15" y1="45.4" x2="117.91" y2="35.73" width="0" layer="19" extent="1-1"/>
+<wire x1="-121.88" y1="-272.81" x2="117.91" y2="35.73" width="0" layer="19" extent="1-1"/>
 </signal>
 <signal name="MCU_TO_RASPI_RESET">
@@
 <signal name="PP5V0_CHG_IN">
 <contactref element="C301" pad="1"/>
-<contactref element="U301" pad="4"/>
 <contactref element="J301" pad="1"/>
 <contactref element="R303" pad="2"/>
@@
 <contactref element="J302" pad="1"/>
 <contactref element="R403" pad="1"/>
-<wire x1="119.51" y1="38.06" x2="122.15" y2="43.5" width="0" layer="19" extent="1-1"/>
+<contactref element="U301" pad="4"/>
 <wire x1="113.13" y1="41.09" x2="119.51" y2="38.06" width="0" layer="19" extent="1-1"/>
 <wire x1="109.94" y1="36.34" x2="113.13" y2="41.09" width="0" layer="19" extent="1-1"/>
@@
 <wire x1="8.12" y1="76.365" x2="109.94" y2="36.34" width="0" layer="19" extent="1-1"/>
 <wire x1="-118.45" y1="-264.85" x2="8.12" y2="76.365" width="0" layer="19" extent="1-1"/>
+<wire x1="-121.88" y1="-274.71" x2="-118.45" y2="-264.85" width="0" layer="19" extent="1-1"/>
 </signal>
 <signal name="3V3_HAT_PG">

Commit message: added battery input jumper
Parts:
- added J402: MOL-SL-2-V, daqcs:MOLSL-2-V
- R401: value 0.05 -> 0.0; device daqcs:RS1206 -> daqcs:R0805
- R402: value 0.0 -> 0.05; device daqcs:R0805 -> daqcs:RS1206
- moved R401 380.8 mm to (-121.7, -263.8)
- moved R402 380.8 mm to (18.2, 90.4)
- moved TP403 379.7 mm to (38.5, 90.2)
- moved TP404 370.2 mm to (-118.5, -255.5)
- moved TP402 22.6 mm to (52.8, 72.6)
Connections:
- new net VBAT_J: J402.1, R402.2A
- net GND: now also TP404.TP; no longer TP403.TP
- net PP3V3_HAT: now also R401.2, TP402.TP; no longer R402.2, TP404.TP
- net PP3V3_LDO: now also R401.1; no longer R402.1
- net VBAT: now also J402.2; no longer R401.2A
- net VBAT_R: now also R402.1A, TP403.TP; no longer R401.1A, TP402.TP
- net VBAT_SNS_N: now also R402.1V; no longer R401.1V
- net VBAT_SNS_P: now also R402.2V; no longer R401.2V

Commit message: added 50mA fuse to external temperature sensor supply line
Parts:
- added F601: FUSE-50MA, daqcs:R0603
- R611: value 0.0 -> 4.7k
- R613: value 4.7k -> 0.0
- moved C602 393.6 mm to (-124.0, -296.5)
- moved R611 36.0 mm to (50.7, 53.8)
- moved R613 34.2 mm to (36.2, 84.7)
- moved R612 3.68 mm to (32.5, 84.8)
Connections:
- new net PP3V3_TEMP: C602.1, F601.1, J605.1, R611.2
- net MCU_TO_BST_RESET: now also R612.2; no longer R611.2
- net MCU_TO_HAT_RESET: now also R613.1; no longer R611.1
- net MCU_TO_RASPI_RESET: now also R613.2; no longer R612.2
- net PP3V3_HAT: now also F601.2; no longer C602.1, J605.1, R613.2
- net TEMP_1WIRE_BI: now also R611.1; no longer R613.1

Commit message: changed sense resistor value to 0.033
Parts:
- added BOM727: SL 70066 2PIN HOUSING, daqcs:BLANK
- added BOM728, BOM729: SL 70058 GOLD CRIMP, daqcs:BLANK
- R402: value 0.05 -> 0.033
- moved R402 422.4 mm to (-122.2, -308.0)
- moved J402 326.0 mm to (2.62, 18.9), turned to 270 degrees
Connections:
- net VBAT_J: now also R402.1A; no longer R402.2A
- net VBAT_R: now also R402.2A; no longer R402.1A
- net VBAT_SNS_N: now also R402.2V; no longer R402.1V
- net VBAT_SNS_P: now also R402.1V; no longer R402.2V

Commit message: removed zeners
Parts:
- J604: value RECEPTACLE-2x3-2.54MM -> MOL-SL-3-V; device daqcs:RECEPTACLE-2X3-254MM -> daqcs:MOLSL-3-V
- J605: value MOL-SL-3-V -> RECEPTACLE-2x3-2.54MM; device daqcs:MOLSL-3-V -> daqcs:RECEPTACLE-2X3-254MM
- R611: value 4.7k -> 0.0
- R613: value 0.0 -> 4.7k
- moved R611 36.0 mm to (32.5, 84.8)
- moved R613 34.2 mm to (50.7, 53.8)
- moved J604 20.2 mm to (54.7, 59.8), turned to 180 degrees
- moved J605 20.2 mm to (34.5, 58.7), turned to 270 degrees
- moved R612 3.68 mm to (36.2, 84.7)
Connections:
- net GND: now also J604.3, J605.4, J605.5; no longer J604.4, J604.5, J605.3
- net MCU_TO_BST_RESET: now also R611.2; no longer R612.2
- net MCU_TO_HAT_RESET: now also R611.1; no longer R613.1
- net MCU_TO_RASPI_RESET: now also R612.2; no longer R613.2
- net PP3V3_TEMP: now also J604.1, R613.2; no longer J605.1, R611.2
- net RASPI_GPIO20: now also J605.1; no longer J604.1
- net RASPI_GPIO26: now also J605.3; no longer J604.3
- net RASPI_RESET_N: now also J605.6; no longer J604.6
- net TEMP_1WIRE_BI: now also J604.2, R613.1; no longer J605.2, R611.1
- net WDT_PET_R: now also J605.2; no longer J604.2
