File: eagle/projects/raspi_cam_adapt/raspi_cam_adapt.sch (EAGLE design)
At the start: 4 parts, among them J201 FFC-FPC-15POS, J202 FFC-FPC-15POS, J203 FFC-FPC-15POS

Commit message: finalized panels
Parts:
- removed LOGO1: (no value), daqcs:CMS_LOGO
- added H201, H202: 2.75mm_drill_3.00mm_radius, daqcs:MOUNT-HOLE_2.75_3.0
- added LOGO201: (no value), daqcs:CMS_LOGO
- J201: value FFC-FPC-15POS -> FFC-FPC-15POS-BOT; device daqcs:FFC-FPC-15POS_FFC15 -> daqcs:FFC-FPC-15POS_FFC15_BOT_SMT
- J202, J203: value FFC-FPC-15POS -> FFC-FPC-15POS-TOP; device daqcs:FFC-FPC-15POS_FFC15 -> daqcs:FFC-FPC-15POS_FFC15_SMT
Other:
- note added: "BOTTOM RIGHT (TOP CONTACTS)"
- note added: "Option 1: - Use a Type 1 FFC/FPC cable (opposite side conductors) - Connect RasPi Zero to J201 - Connect Type 1 cable to J202 Option 2: - Use a Type 2 FFC/FPC cable (same side conductors) - Connect RasPi Zero to J201 - Connect Type 1 cable to J203 *Note that FFC/FPC cable contacts face towards the RasPi Zero board and Camera Module when connecting. FFC-FPC 15PIN 1MM PITCH CONNECTOR Bottom Cotacts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"
- note added: "TOP LEFT (BOTTOM CONTACTS)"
- note added: "TOP RIGHT (TOP CONTACTS)"
- note removed: "BOTTOM RIGHT"
- note removed: "Option 1: - Use a Type 1 FFC/FPC cable (opposite side conductors) - Connect RasPi Zero to J201 - Connect Type 1 cable to J203 Option 2: - Use a Type 2 FFC/FPC cable (same side conductors) - Connect RasPi Zero to J201 - Connect Type 1 cable to J202 *Note that FFC/FPC cable contacts face towards the RasPi Zero board and Camera Module when connecting. FFC-FPC 15PIN 1MM PITCH CONNECTOR (J201, J202, J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"
- note removed: "TOP LEFT"
- note removed: "TOP RIGHT"
Changed lines of the file:
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@@
 </attributes>
 <variantdefs>
+<variantdef name="POR"/>
 </variantdefs>
 <classes>
@@
 <part name="FRAME101" library="daqcs" deviceset="FRAME_B_L" device=""/>
 <part name="FRAME201" library="daqcs" deviceset="FRAME_B_L" device=""/>
-<part name="J201" library="daqcs" deviceset="FFC-FPC-15POS" device="" technology="_FFC15" value="FFC-FPC-15POS"/>
-<part name="J203" library="daqcs" deviceset="FFC-FPC-15POS" device="" technology="_FFC15" value="FFC-FPC-15POS"/>
+<part name="J201" library="daqcs" deviceset="FFC-FPC-15POS" device="_SMT" technology="_FFC15_BOT" value="FFC-FPC-15POS-BOT"/>
+<part name="J203" library="daqcs" deviceset="FFC-FPC-15POS" device="_SMT" technology="_FFC15" value="FFC-FPC-15POS-TOP">
+<variant name="POR" populate="no"/>
+</part>
 <part name="TOC101" library="daqcs" deviceset="TOC-10" device=""/>
-<part name="J202" library="daqcs" deviceset="FFC-FPC-15POS" device="" technology="_FFC15" value="FFC-FPC-15POS"/>
-<part name="LOGO1" library="daqcs" deviceset="CMS_LOGO" device=""/>
+<part name="J202" library="daqcs" deviceset="FFC-FPC-15POS" device="_SMT" technology="_FFC15" value="FFC-FPC-15POS-TOP"/>
+<part name="LOGO201" library="daqcs" deviceset="CMS_LOGO" device=""/>
+<part name="H201" library="daqcs" deviceset="MOUNT-HOLE" device="_2.75_3.0" value="2.75mm_drill_3.00mm_radius"/>
+<part name="H202" library="daqcs" deviceset="MOUNT-HOLE" device="_2.75_3.0" value="2.75mm_drill_3.00mm_radius"/>
 </parts>
 <sheets>
@@
 <plain>
 <text x="124.46" y="251.46" size="11.43" layer="91">FFC-FPC CONNECTORS</text>
-<text x="22.86" y="68.58" size="3.81" layer="91" rot="R90">TOP LEFT</text>
-<text x="213.36" y="63.5" size="3.81" layer="91" rot="R90">BOTTOM RIGHT</text>
-<text x="210.82" y="170.18" size="3.81" layer="91" rot="R90">TOP RIGHT</text>
+<text x="15.24" y="81.28" size="3.81" layer="91" rot="R90" align="center">TOP LEFT
+(BOTTOM CONTACTS)</text>
+<text x="213.36" y="81.28" size="3.81" layer="91" rot="R90" align="center">BOTTOM RIGHT
+(TOP CONTACTS)</text>
+<text x="210.82" y="182.88" size="3.81" layer="91" rot="R90" align="center">TOP RIGHT
+(TOP CONTACTS)</text>
 <text x="233.68" y="215.9" size="6.35" layer="91">Connection Options:</text>
-<text x="236.22" y="106.68" size="3.81" layer="91">Option 1:
+<text x="238.76" y="76.2" size="3.81" layer="91">Option 1:
 - Use a Type 1 FFC/FPC cable (opposite side conductors)
 - Connect RasPi Zero to J201
-- Connect Type 1 cable to J203
+- Connect Type 1 cable to J202
 Option 2:
 - Use a Type 2 FFC/FPC cable (same side conductors)
 - Connect RasPi Zero to J201
-- Connect Type 1 cable to J202
+- Connect Type 1 cable to J203
 *Note that FFC/FPC cable contacts face towards the RasPi
 Zero board and Camera Module when connecting.
-FFC-FPC 15PIN 1MM PITCH CONNECTOR (J201, J202, J203)
-Manufacturer: Amphenol FCI
-Manufacturer PN: SFW15R-2STE1LF
-Vendor: Digi-Key
-Vendor PN: 609-1906-1-ND </text>
+FFC-FPC 15PIN 1MM PITCH CONNECTOR
+  Bottom Cotacts (J201)
+    Manufacturer: Amphenol FCI
+    Manufacturer PN: SFW15R-1STE1LF
+    Vendor: Digi-Key
+    Vendor PN: 609-1905-1-ND
+  Top Cotacts (J202,J203)
+    Manufacturer: Amphenol FCI
+    Manufacturer PN: SFW15R-2STE1LF
+    Vendor: Digi-Key
+    Vendor PN: 609-1906-1-ND </text>
 <text x="330.2" y="27.94" size="3.81" layer="91">CONNECTORS</text>
 <text x="421.64" y="7.62" size="3.81" layer="91">1</text>
@@
 <instance part="J203" gate="G$1" x="198.12" y="78.74" rot="MR0"/>
 <instance part="J202" gate="G$1" x="198.12" y="182.88" rot="MR0"/>
-<instance part="LOGO1" gate="G$1" x="276.86" y="60.96"/>
+<instance part="LOGO201" gate="G$1" x="238.76" y="20.32"/>
+<instance part="H201" gate="G$1" x="274.32" y="30.48"/>
+<instance part="H202" gate="G$1" x="274.32" y="20.32"/>
 </instances>
 <busses>

Commit message: removed inner pours on camera adapte board, re-panneled
Parts:
- removed J203: FFC-FPC-15POS-TOP, daqcs:FFC-FPC-15POS_FFC15_SMT
Connections:
- removed net GND: J201.1, J201.10, J201.4, J201.7, J202.12, J202.15, J202.6, J202.9, J203.1, J203.10, J203.4, J203.7
- new net GND_1: J201.1, J202.15
- new net GND_2: J201.4, J202.12
- new net GND_3: J201.7, J202.9
- new net GND_4: J201.10, J202.6
- net 3V3: no longer J203.15
- net CAM1_CN: no longer J203.8
- net CAM1_CP: no longer J203.9
- net CAM1_DN0: no longer J203.2
- net CAM1_DN1: no longer J203.5
- net CAM1_DP0: no longer J203.3
- net CAM1_DP1: no longer J203.6
- net CAM_GPIO0: no longer J203.11
- net CAM_GPIO1: no longer J203.12
- net SCL0: no longer J203.13
- net SDA0: no longer J203.14
Other:
- note added: "Option 1: - Use a Type 1 FFC/FPC cable (opposite side conductors) - Connect RasPi Zero to J201 - Connect Type 1 cable to J202 (which is a top-side contact connector) Option 2: - Use a Type 2 FFC/FPC cable (same side conductors) - Connect RasPi Zero to J201 - Connect Type 1 cable to J202 (which is a bottom-side contact connector) *Note that FFC/FPC cable contacts face towards the RasPi Zero board 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"
- note added: "TOP LEFT"
- note added: "TOP RIGHT"
- note removed: "BOTTOM RIGHT (TOP CONTACTS)"
- note removed: "Option 1: - Use a Type 1 FFC/FPC cable (opposite side conductors) - Connect RasPi Zero to J201 - Connect Type 1 cable to J202 Option 2: - Use a Type 2 FFC/FPC cable (same side conductors) - Connect RasPi Zero to J201 - Connect Type 1 cable to J203 *Note that FFC/FPC cable contacts face towards the RasPi Zero board and Camera Module when connecting. FFC-FPC 15PIN 1MM PITCH CONNECTOR Bottom Cotacts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"
- note removed: "TOP LEFT (BOTTOM CONTACTS)"
- note removed: "TOP RIGHT (TOP CONTACTS)"
